File: mainboard/MainShutdown.sch (KiCad schematic (older format))
At the start: 50 parts, among them J5 AIR-, J6 AIR+, K1 KT12-1A, Q1 TSM2306, Q10 TSM3401, Q11 TSM3401, Q12 TSM2306, Q13 TSM2312, Q14 BC846AW, Q2 TSM3401, Q3 TSM3401, Q4 TSM3401, Q5 TSM2306, Q6 TSM2306, Q7 TSM3401, Q8 TSM2312, Q9 TSM3401, U11 MAX16053, U12 SN74LVC1G123

Commit message: Shutdown logic to use gates, changed mosfets
Shutdown ported from new car, mosfets changed to higher VGS max
Parts:
- removed D3: BT150S-600R, MainBoard:TO-252-2, symbol Device:Q_SCR_KAG
- added C19, C27, C29, C30: 100n, Capacitor_SMD:C_0805_2012Metric, symbol Device:C
- added D3: 12V, symbol Device:D_Zener
- added D8: 1N4148, Diode_THT:D_DO-35_SOD27_P7.62mm_Horizontal, symbol Diode:1N4148
- added K2: UMS05-1A80-75L, MainBoard:G6DN-1A_DC12, symbol Relay:UMS05-1A80-75L
- added Q17: SSM3K361TU,LF, symbol Device:Q_NMOS_GSD
- added Q18, Q19, Q20: NTR4003, Package_TO_SOT_SMD:SOT-23, symbol Device:Q_NMOS_GSD
- added R60, R61, R64, R66: 10k, Resistor_SMD:R_0805_2012Metric, symbol Device:R
- added R62, R63, R65: 10, Resistor_SMD:R_0805_2012Metric, symbol Device:R
- added U13: LM339, symbol Comparator:LM339
- added U16: 4044, symbol 4xxx_IEEE:4044
- added U21: 4082, symbol 4xxx_IEEE:4082
- D4: value MMBZ4624 -> MMBZ4624 4V7
- Q1: value TSM2306 -> NTR4003
- R15: value 100K -> 1M
Connections:
- net +12V: now also C19.1, C29.1, C30.1, D8.1 (K), K2.2, R64.1, U13.3 (V+), U16.16 (Vdd), U16.5 (EN), U21.14 (Vdd), U21.14 (Vdd)
- net +3V3: now also R60.1
- net BMS_LED: now also Q19.3 (D)
- net BMS_Status: now also U13.5 (+)
- net From_SD: now also R15.1, K2.3
- net From_TSMS: no longer Q1.1 (G), R15.1
- net GND: now also C19.2, C27.2, C29.2, C30.2, D3.2 (A), Q17.2 (S), Q18.2 (S), Q19.2 (S), Q20.2 (S), R61.2, R66.1, U13.12 (V-), U16.8 (Vss), U21.7 (Vss), U21.7 (Vss); no longer R15.2
- net IMD_LED: now also Q18.3 (D)
- net IMD_Status: now also U16.12
- net TS_ON: now also U13.7 (+)
- net To_TSMS: now also K2.4
- net ~RESET: now also U16.11, U16.7
- net at D4.1 (K), J6.2 (Pin_2): now also Q17.3 (D)
- net at R31.1, R33.1: now also Q17.1 (G)
- new net: D3.1 (K), Q1.1 (G), R15.2
- new net: U13.2, U16.6
- new net: U13.1, U21.9
- new net: R64.2, U21.12
- new net: R65.2, U21.13
- new net: Q20.1 (G), R65.1, R66.2
- new net: D8.2 (A), K2.1, Q20.3 (D)
- new net: Q18.1 (G), R62.1
- new net: Q19.1 (G), R63.1
- new net 1V5_REF: C27.1, R60.2, R61.1, U13.10 (-), U13.4 (-), U13.6 (-), U13.8 (-)
- new net BMS_LATCHED: R63.2, U16.9, U21.10
- new net IMD_LATCHED: R62.2, U16.10, U21.11
- no-connect marks 0 -> 6
Other:
- note added: "12V CMOS\nHIGH: OK\nLOW: fault"
- note added: "3V3 uC\nHIGH: OK\nLOW: fault"
- note added: "Actual daisychain connection \nof the shutdown line"
- note added: "CHECK: unpopulated"
- note added: "Latching mechanism"
- note added: "Let the uC know the status \nof the shutdown before"
- note added: "Power supply controller, gives a delay on \n~RESET~ line after reset event."
- note added: "R64 can be used to \nmanually test shutdown"
- note added: "TODO: check this section, it may not be\n needed since TS_ON will go straight to the AND"
- note added: "if\nB: rising edge\nthen\nQ: square pulse"
- moved on the sheet: C23, C24, D1, D2, D4, J5, J6, K1, Q1, Q10, Q11, Q12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

Commit message: ported shutdown from new car
Parts:
- removed C24: 10n, Capacitor_SMD:C_0805_2012Metric, symbol Device:C
- removed D1: BT150S-600R, MainBoard:TO-252-2, symbol Device:Q_SCR_KAG
- removed Q10, Q11, Q2, Q3, Q4, Q7, Q9: TSM3401, Package_TO_SOT_SMD:SOT-23, symbol Device:Q_PMOS_GSD
- removed Q12, Q5, Q6: TSM2306, Package_TO_SOT_SMD:SOT-23, symbol Device:Q_NMOS_GSD
- removed Q13, Q8: TSM2312, Package_TO_SOT_SMD:SOT-23, symbol Device:Q_NMOS_GSD
- removed R12, R23: 1M, Resistor_SMD:R_0805_2012Metric, symbol Device:R
- removed R16, R17, R19, R24, R25, R28: 10K, Resistor_SMD:R_0805_2012Metric, symbol Device:R
- removed R20: 2K2, Resistor_SMD:R_0805_2012Metric, symbol Device:R
- removed R21, R22, R27, R29: 100K, Resistor_SMD:R_0805_2012Metric, symbol Device:R
- removed R26: 3.3K, Resistor_SMD:R_0805_2012Metric, symbol Device:R
- removed U12: SN74LVC1G123, Package_SO:VSSOP-8_2.3x2mm_P0.5mm, symbol MainBoard:SN74LVC1G123
Connections:
- net From_SD: now also K2.4; no longer K2.3
- net To_TSMS: now also K2.3; no longer K2.4
Other:
- note added: "AIRs have internal suppression mechanisms \nthat clips output to 55V, \ndon't place outside suppression."
- note added: "AIRs needs no other suppression \nmechanism, populate diode \nonly if they're disconnected."
- note removed: "BMS_SHUTDOWN"
- note removed: "IMD_SHUTDOWN"
- note removed: "TODO: check this section, it may not be\n needed since TS_ON will go straight to the AND"
- note removed: "TRACTIVE SYSTEM CONTROL"
- note removed: "do not populate\nflyback diode if\nnot strictly necessary"
- note removed: "if\nB: rising edge\nthen\nQ: square pulse"
- moved on the sheet: C30, D4, J5, J6, Q17, R31, R33, U21A
