File: mainboard/MainShutdown.sch (KiCad schematic (older format))
At the start: 41 parts, among them J5 AIR-, J6 AIR+, K1 KT12-1A, K2 UMS05-1A80-75L, Q1 NTR4003, Q14 BC846AW, Q17 SSM3K361TU,LF, Q18 NTR4003, Q19 NTR4003, Q20 NTR4003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

Commit message: finished footprint association
Parts:
- D8: value 1N4148 -> BAS16GW; footprint Diode_THT:D_DO-35_SOD27_P7.62mm_Horizontal -> Diode_SMD:D_SOD-123
- DZ3: renamed from D3; value 12V -> MMBZ4624 4V7; footprint (none) -> Diode_SMD:D_SOT-23_ANK
- Q1, Q18, Q19, Q20: value NTR4003 -> TSM2306
- Q17: value SSM3K361TU,LF -> IRLML0100TRPbF; footprint (none) -> Package_TO_SOT_SMD:SOT-23
- R11, R14, R33: value 100K -> 100k
- R13: value 220K -> 220k
- R18, R34, R35: value 10K -> 10k
- R30: value 1K -> 1k
- R31: value 3.3K -> 3.3k
- R32: value 22K -> 22k
- U13: value LM339 -> TS3704IPT; footprint (none) -> Package_SO:TSSOP-14_4.4x5mm_P0.65mm
- U16: value 4044 -> CD4044; footprint (none) -> Package_SO:TSSOP-16_4.4x5mm_P0.65mm
- U21: value 4082 -> CD4082; footprint (none) -> Package_SO:TSSOP-14_4.4x5mm_P0.65mm
- renumbered D4 to DZ4
Changed lines of the file:
@@
 P 1000 1300
 F 0 "R14" V 900 1300 50  0000 C CNN
-F 1 "100K" V 1000 1300 50  0000 C CNN
+F 1 "100k" V 1000 1300 50  0000 C CNN
 F 2 "Resistor_SMD:R_0805_2012Metric" V 930 1300 50  0001 C CNN
 F 3 "~" H 1000 1300 50  0001 C CNN
@@
 P 700 1300
 F 0 "R13" V 600 1300 50  0000 C CNN
-F 1 "220K" V 700 1300 50  0000 C CNN
+F 1 "220k" V 700 1300 50  0000 C CNN
 F 2 "Resistor_SMD:R_0805_2012Metric" V 630 1300 50  0001 C CNN
 F 3 "~" H 700 1300 50  0001 C CNN
@@
 P 700 1900
 F 0 "R18" V 600 1900 50  0000 C CNN
-F 1 "10K" V 700 1900 50  0000 C CNN
+F 1 "10k" V 700 1900 50  0000 C CNN
 F 2 "Resistor_SMD:R_0805_2012Metric" V 630 1900 50  0001 C CNN
 F 3 "~" H 700 1900 50  0001 C CNN
@@
 P 6400 7400
 F 0 "R34" V 6300 7400 50  0000 C CNN
-F 1 "10K" V 6400 7400 50  0000 C CNN
+F 1 "10k" V 6400 7400 50  0000 C CNN
 F 2 "MainBoard:TO-247_wHeatsink" V 6330 7400 50  0001 C CNN
 F 3 "~" H 6400 7400 50  0001 C CNN
@@
 P 6700 7400
 F 0 "R35" V 6600 7400 50  0000 C CNN
-F 1 "10K" V 6700 7400 50  0000 C CNN
+F 1 "10k" V 6700 7400 50  0000 C CNN
 F 2 "MainBoard:TO-247_wHeatsink" V 6630 7400 50  0001 C CNN
 F 3 "~" H 6700 7400 50  0001 C CNN
@@
 P 1450 7400
 F 0 "R33" V 1350 7400 50  0000 C CNN
-F 1 "100K" V 1450 7400 50  0000 C CNN
+F 1 "100k" V 1450 7400 50  0000 C CNN
 F 2 "Resistor_SMD:R_0805_2012Metric" V 1380 7400 50  0001 C CNN
 F 3 "~" H 1450 7400 50  0001 C CNN
@@
 P 1200 7250
 F 0 "R31" V 1100 7250 50  0000 C CNN
-F 1 "3.3K" V 1200 7250 50  0000 C CNN
+F 1 "3.3k" V 1200 7250 50  0000 C CNN
 F 2 "Resistor_SMD:R_0805_2012Metric" V 1130 7250 50  0001 C CNN
 F 3 "~" H 1200 7250 50  0001 C CNN
@@
 P 3500 7150
 F 0 "R32" V 3400 7150 50  0000 C CNN
-F 1 "22K" V 3500 7150 50  0000 C CNN
+F 1 "22k" V 3500 7150 50  0000 C CNN
 F 2 "Resistor_SMD:R_0805_2012Metric" V 3430 7150 50  0001 C CNN
 F 3 "~" H 3500 7150 50  0001 C CNN
@@
 P 4050 6700
 F 0 "R30" V 3950 6700 50  0000 C CNN
-F 1 "1K" V 4050 6700 50  0000 C CNN
+F 1 "1k" V 4050 6700 50  0000 C CNN
 F 2 "Resistor_SMD:R_0805_2012Metric" V 3980 6700 50  0001 C CNN
 F 3 "~" H 4050 6700 50  0001 C CNN
@@
 $EndComp
 $Comp
-L Device:D_Zener D4
+L Device:D_Zener DZ4
 U 1 1 5B0DE15E
 P 2650 7150
-F 0 "D4" H 2650 7050 50  0000 C CNN
+F 0 "DZ4" H 2650 7050 50  0000 C CNN
 F 1 "MMBZ4624 4V7" H 2650 7250 50  0000 C CNN
 F 2 "Diode_SMD:D_SOT-23_ANK" H 2650 7150 50  0001 C CNN
@@
 P 2900 1050
 F 0 "R11" V 2800 1050 50  0000 C CNN
-F 1 "100K" V 2900 1050 50  0000 C CNN
+F 1 "100k" V 2900 1050 50  0000 C CNN
 F 2 "Resistor_SMD:R_0805_2012Metric" V 2830 1050 50  0001 C CNN
 F 3 "~" H 2900 1050 50  0001 C CNN
@@
 P 1750 5450
 F 0 "Q1" H 1950 5500 50  0000 L CNN
-F 1 "NTR4003" H 1950 5400 50  0000 L CNN
+F 1 "TSM2306" H 1950 5400 50  0000 L CNN
 F 2 "Package_TO_SOT_SMD:SOT-23" H 1950 5550 50  0001 C CNN
 F 3 "http://www.taiwansemi.com/products/datasheet/TSM2306_B15.pdf" H 1750 5450 50  0001 C CNN
@@
 $EndComp
 $Comp
-L Device:D_Zener D3
+L Device:D_Zener DZ3
 U 1 1 603F2A0C
 P 1450 5700
-F 0 "D3" V 1404 5780 50  0000 L CNN
-F 1 "12V" V 1495 5780 50  0000 L CNN
-F 2 "" H 1450 5700 50  0001 C CNN
-F 3 "~" H 1450 5700 50  0001 C CNN
+F 0 "DZ3" V 1404 5780 50  0000 L CNN
+F 1 "MMBZ4624 4V7" V 1495 5780 50  0000 L CNN
+F 2 "Diode_SMD:D_SOT-23_ANK" H 1450 5700 50  0001 C CNN
+F 3 "http://www.vishay.com/docs/85770/mmbz4617.pdf" H 1450 5700 50  0001 C CNN
 	1    1450 5700
 	0    1    1    0
@@
 P 1750 7250
 F 0 "Q17" H 1954 7296 50  0000 L CNN
-F 1 "SSM3K361TU,LF" H 1954 7205 50  0000 L CNN
-F 2 "" H 1950 7350 50  0001 C CNN
-F 3 "~" H 1750 7250 50  0001 C CNN
+F 1 "IRLML0100TRPbF" H 1954 7205 50  0000 L CNN
+F 2 "Package_TO_SOT_SMD:SOT-23" H 1950 7350 50  0001 C CNN
+F 3 "https://www.mouser.it/datasheet/2/196/irlml0100pbf-1228126.pdf" H 1750 7250 50  0001 C CNN
 	1    1750 7250
 	1    0    0    -1
@@
 P 4900 3450
 F 0 "U16" H 4750 4000 50  0000 C CNN
-F 1 "4044" H 4750 3900 50  0000 C CNN
-F 2 "" H 4900 3450 50  0001 C CNN
+F 1 "CD4044" H 4750 3900 50  0000 C CNN
+F 2 "Package_SO:TSSOP-16_4.4x5mm_P0.65mm" H 4900 3450 50  0001 C CNN
 F 3 "" H 4900 3450 50  0001 C CNN
 	1    4900 3450
@@
 P 8650 3500
 F 0 "U21" H 8450 3900 50  0000 C CNN
-F 1 "4082" H 8450 3800 50  0000 C CNN
-F 2 "" H 8650 3500 50  0001 C CNN
+F 1 "CD4082" H 8450 3800 50  0000 C CNN
+F 2 "Package_SO:TSSOP-14_4.4x5mm_P0.65mm" H 8650 3500 50  0001 C CNN
 F 3 "" H 8650 3500 50  0001 C CNN
 	2    8650 3500
@@
 P 6750 950
 F 0 "U21" H 6600 1200 50  0000 C CNN
-F 1 "4082" H 6900 1200 50  0000 C CNN
-F 2 "" H 6750 950 50  0001 C CNN
+F 1 "CD4082" H 6900 1200 50  0000 C CNN
+F 2 "Package_SO:TSSOP-14_4.4x5mm_P0.65mm" H 6750 950 50  0001 C CNN
 F 3 "" H 6750 950 50  0001 C CNN
 	1    6750 950
@@
 P 3500 3750
 F 0 "U13" H 3500 4117 50  0000 C CNN
-F 1 "LM339" H 3500 4026 50  0000 C CNN
-F 2 "" H 3450 3850 50  0001 C CNN
+F 1 "TS3704IPT" H 3500 4026 50  0000 C CNN
+F 2 "Package_SO:TSSOP-14_4.4x5mm_P0.65mm" H 3450 3850 50  0001 C CNN
 F 3 "https://www.st.com/resource/en/datasheet/lm139.pdf" H 3550 3950 50  0001 C CNN
 	1    3500 3750
@@
 P 7350 3350
 F 0 "U13" H 7350 3717 50  0000 C CNN
-F 1 "LM339" H 7350 3626 50  0000 C CNN
-F 2 "" H 7300 3450 50  0001 C CNN
+F 1 "TS3704IPT" H 7350 3626 50  0000 C CNN
+F 2 "Package_SO:TSSOP-14_4.4x5mm_P0.65mm" H 7300 3450 50  0001 C CNN
 F 3 "https://www.st.com/resource/en/datasheet/lm139.pdf" H 7400 3550 50  0001 C CNN
 	2    7350 3350
@@
 P 4400 1250
 F 0 "U13" H 4400 1617 50  0000 C CNN
-F 1 "LM339" H 4400 1526 50  0000 C CNN
-F 2 "" H 4350 1350 50  0001 C CNN
+F 1 "TS3704IPT" H 4400 1526 50  0000 C CNN
+F 2 "Package_SO:TSSOP-14_4.4x5mm_P0.65mm" H 4350 1350 50  0001 C CNN
 F 3 "https://www.st.com/resource/en/datasheet/lm139.pdf" H 4450 1450 50  0001 C CNN
 	3    4400 1250
@@
 P 5400 1250
 F 0 "U13" H 5400 1617 50  0000 C CNN
-F 1 "LM339" H 5400 1526 50  0000 C CNN
-F 2 "" H 5350 1350 50  0001 C CNN
+F 1 "TS3704IPT" H 5400 1526 50  0000 C CNN
+F 2 "Package_SO:TSSOP-14_4.4x5mm_P0.65mm" H 5350 1350 50  0001 C CNN
 F 3 "https://www.st.com/resource/en/datasheet/lm139.pdf" H 5450 1450 50  0001 C CNN
 	4    5400 1250
@@
 P 1000 3500
 F 0 "U13" H 958 3546 50  0000 L CNN
-F 1 "LM339" H 958 3455 50  0000 L CNN
-F 2 "" H 950 3600 50  0001 C CNN
+F 1 "TS3704IPT" H 958 3455 50  0000 L CNN
+F 2 "Package_SO:TSSOP-14_4.4x5mm_P0.65mm" H 950 3600 50  0001 C CNN
 F 3 "https://www.st.com/resource/en/datasheet/lm139.pdf" H 1050 3700 50  0001 C CNN
 	5    1000 3500
@@
 P 9550 2900
 F 0 "D8" V 9500 3050 50  0000 R CNN
-F 1 "1N4148" V 9600 3250 50  0000 R CNN
-F 2 "Diode_THT:D_DO-35_SOD27_P7.62mm_Horizontal" H 9550 2725 50  0001 C CNN
-F 3 "https://assets.nexperia.com/documents/data-sheet/1N4148_1N4448.pdf" H 9550 2900 50  0001 C CNN
+F 1 "BAS16GW" V 9600 3250 50  0000 R CNN
+F 2 "Diode_SMD:D_SOD-123" H 9550 2725 50  0001 C CNN
+F 3 "https://assets.nexperia.com/documents/data-sheet/BAS16GW.pdf" H 9550 2900 50  0001 C CNN
 	1    9550 2900
 	0    -1   1    0
@@
 P 9750 3500
 F 0 "Q20" H 9950 3550 50  0000 L CNN
-F 1 "NTR4003" H 9950 3450 50  0000 L CNN
+F 1 "TSM2306" H 9950 3450 50  0000 L CNN
 F 2 "Package_TO_SOT_SMD:SOT-23" H 9950 3600 50  0001 C CNN
 F 3 "http://www.taiwansemi.com/products/datasheet/TSM2306_B15.pdf" H 9750 3500 50  0001 C CNN
@@
 P 5700 4850
 F 0 "Q18" H 5900 4900 50  0000 L CNN
-F 1 "NTR4003" H 5900 4800 50  0000 L CNN
+F 1 "TSM2306" H 5900 4800 50  0000 L CNN
 F 2 "Package_TO_SOT_SMD:SOT-23" H 5900 4950 50  0001 C CNN
 F 3 "http://www.taiwansemi.com/products/datasheet/TSM2306_B15.pdf" H 5700 4850 50  0001 C CNN
@@
 P 6600 4900
 F 0 "Q19" H 6800 4950 50  0000 L CNN
-F 1 "NTR4003" H 6800 4850 50  0000 L CNN
+F 1 "TSM2306" H 6800 4850 50  0000 L CNN
 F 2 "Package_TO_SOT_SMD:SOT-23" H 6800 5000 50  0001 C CNN
 F 3 "http://www.taiwansemi.com/products/datasheet/TSM2306_B15.pdf" H 6600 4900 50  0001 C CNN

Commit message: Done early board
Parts:
- removed R34, R35: 10k, MainBoard:TO-247_wHeatsink, symbol Device:R
- added R20: PWR163S-25-1002J 10k, MainBoard:pwr163, symbol MainBoard:R_power_backplane
Connections:
- net +BATT: now also K1.4; no longer K1.3
- net +TS: now also R20.2
- net BMS_LATCHED: now also U21.11; no longer U21.10
- net IMD_LATCHED: now also U21.10; no longer U21.11
- new net: K1.3, R20.1
- new net R20_heatsink: R20.3 (back)
Other:
- note removed: "AP101 10K"
Changed lines of the file:
@@
 encoding utf-8
 Sheet 2 3
-Title "Chimera BMS"
-Date "2021-03-28"
+Title "Chimera BMS - MainBoard"
+Date "2021-03-29"
 Rev "V3"
 Comp "E-Agle TRT"
@@
 	1    0    0    -1
 $EndComp
-Wire Wire Line
-	6300 7150 6400 7150
 $Comp
 L power:GND #PWR093
@@
 $EndComp
 $Comp
-L Device:R R34
-U 1 1 5B0DE0DA
-P 6400 7400
-F 0 "R34" V 6300 7400 50  0000 C CNN
-F 1 "10k" V 6400 7400 50  0000 C CNN
-F 2 "MainBoard:TO-247_wHeatsink" V 6330 7400 50  0001 C CNN
-F 3 "~" H 6400 7400 50  0001 C CNN
-	1    6400 7400
-	1    0    0    -1
-$EndComp
-Text Notes 6550 7600 1    50   ~ 0
-AP101 10K
-$Comp
 L MainBoard:+TS #PWR097
 U 1 1 5B0DE0E2
-P 6300 7650
-F 0 "#PWR097" H 6300 7500 50  0001 C CNN
-F 1 "+TS" V 6300 7800 50  0000 L CNN
-F 2 "" H 6200 7400 50  0001 C CNN
-F 3 "" H 6300 7500 50  0001 C CNN
-	1    6300 7650
-	0    -1   -1   0
-$EndComp
-$Comp
-L Device:R R35
-U 1 1 5B0DE0E8
-P 6700 7400
-F 0 "R35" V 6600 7400 50  0000 C CNN
-F 1 "10k" V 6700 7400 50  0000 C CNN
-F 2 "MainBoard:TO-247_wHeatsink" V 6630 7400 50  0001 C CNN
-F 3 "~" H 6700 7400 50  0001 C CNN
-	1    6700 7400
-	1    0    0    -1
+P 6700 6750
+F 0 "#PWR097" H 6700 6600 50  0001 C CNN
+F 1 "+TS" V 6700 6900 50  0000 L CNN
+F 2 "" H 6600 6500 50  0001 C CNN
+F 3 "" H 6700 6600 50  0001 C CNN
+	1    6700 6750
+	0    1    1    0
 $EndComp
 Wire Wire Line
@@
 L power:+BATT #PWR092
 U 1 1 5B0DE0F0
-P 6400 6750
-F 0 "#PWR092" H 6400 6600 50  0001 C CNN
-F 1 "+BATT" V 6400 6900 50  0000 L CNN
-F 2 "" H 6400 6750 50  0001 C CNN
-F 3 "" H 6400 6750 50  0001 C CNN
-	1    6400 6750
+P 6300 7150
+F 0 "#PWR092" H 6300 7000 50  0001 C CNN
+F 1 "+BATT" V 6300 7300 50  0000 L CNN
+F 2 "" H 6300 7150 50  0001 C CNN
+F 3 "" H 6300 7150 50  0001 C CNN
+	1    6300 7150
 	0    1    1    0
 $EndComp
-Wire Wire Line
-	6400 7550 6400 7650
-Wire Wire Line
-	6400 7150 6400 7250
-Connection ~ 6400 7150
 Text Notes 4750 6450 0    50   ~ 0
 PRE-CHARGE CIRCUIT
-Wire Wire Line
-	6300 7650 6400 7650
-Connection ~ 6400 7650
-Wire Wire Line
-	6700 7650 6700 7550
-Wire Wire Line
-	6400 7650 6700 7650
-Wire Wire Line
-	6700 7150 6700 7250
-Wire Wire Line
-	6400 7150 6700 7150
 $Comp
 L Connector_Generic:Conn_01x02 J6
@@
 Text HLabel 7050 3250 0    50   Input ~ 0
 TS_ON
+Text Label 7700 3550 0    50   ~ 0
+BMS_LATCHED
 Text Label 7700 3450 0    50   ~ 0
-BMS_LATCHED
-Text Label 7700 3550 0    50   ~ 0
 IMD_LATCHED
 $Comp
@@
 Text Notes 3550 4250 0    50   ~ 0
 12V CMOS\nHIGH: OK\nLOW: fault
-Text Notes 2700 3600 0    50   ~ 0
-3V3 uC\nHIGH: OK\nLOW: fault
 Wire Wire Line
 	3200 1300 2900 1300
@@
 Text Notes 1100 2200 0    50   ~ 0
 Power supply controller, gives a delay on \n~RESET~ line after reset event.
-$Comp
-L Comparator:LM339 U13
-U 1 1 604E735B
-P 3500 3750
-F 0 "U13" H 3500 4117 50  0000 C CNN
-F 1 "TS3704IPT" H 3500 4026 50  0000 C CNN
-F 2 "Package_SO:TSSOP-14_4.4x5mm_P0.65mm" H 3450 3850 50  0001 C CNN
-F 3 "https://www.st.com/resource/en/datasheet/lm139.pdf" H 3550 3950 50  0001 C CNN
-	1    3500 3750
-	1    0    0    -1
-$EndComp
-$Comp
-L Comparator:LM339 U13
-U 2 1 604E8BD0
-P 7350 3350
-F 0 "U13" H 7350 3717 50  0000 C CNN
-F 1 "TS3704IPT" H 7350 3626 50  0000 C CNN
-F 2 "Package_SO:TSSOP-14_4.4x5mm_P0.65mm" H 7300 3450 50  0001 C CNN
-F 3 "https://www.st.com/resource/en/datasheet/lm139.pdf" H 7400 3550 50  0001 C CNN
-	2    7350 3350
-	1    0    0    -1
-$EndComp
 $Comp
 L Comparator:LM339 U13
@@
 	6700 4650 6750 4650
 Wire Wire Line
+	7700 3550 8150 3550
+Wire Wire Line
 	7700 3450 8150 3450
-Wire Wire Line
-	7700 3550 8150 3550
 Wire Wire Line
 	7650 3350 8150 3350
@@
 Wire Wire Line
 	2800 7150 3350 7150
+$Comp
+L Comparator:LM339 U13
+U 1 1 604E735B
+P 3500 3750
+F 0 "U13" H 3500 4117 50  0000 C CNN
+F 1 "TS3704IPT" H 3500 4026 50  0000 C CNN
+F 2 "Package_SO:TSSOP-14_4.4x5mm_P0.65mm" H 3450 3850 50  0001 C CNN
+F 3 "https://www.st.com/resource/en/datasheet/lm139.pdf" H 3550 3950 50  0001 C CNN
+	1    3500 3750
+	1    0    0    -1
+$EndComp
+Text Notes 2700 3600 0    50   ~ 0
+3V3 uC\nHIGH: OK\nLOW: fault
+$Comp
+L Comparator:LM339 U13
+U 2 1 604E8BD0
+P 7350 3350
+F 0 "U13" H 7350 3717 50  0000 C CNN
+F 1 "TS3704IPT" H 7350 3626 50  0000 C CNN
+F 2 "Package_SO:TSSOP-14_4.4x5mm_P0.65mm" H 7300 3450 50  0001 C CNN
+F 3 "https://www.st.com/resource/en/datasheet/lm139.pdf" H 7400 3550 50  0001 C CNN
+	2    7350 3350
+	1    0    0    -1
+$EndComp
+$Comp
+L MainBoard:R_power_backplane R20
+U 1 1 606B3E8B
+P 6550 6750
+F 0 "R20" H 6620 6750 50  0000 L CNN
+F 1 "PWR163S-25-1002J 10k" V 6700 6750 50  0001 C CNN
+F 2 "MainBoard:pwr163" V 6510 6750 50  0001 C CNN
+F 3 "~" H 6550 6750 50  0001 C CNN
+	1    6550 6750
+	0    -1   -1   0
+$EndComp
+Text Label 6850 7000 3    50   ~ 0
+R20_heatsink
+Wire Wire Line
+	6550 7000 6850 7000
 $EndSCHEMATC

Commit message: board soldered
Parts:
- added R23: 100k, Resistor_SMD:R_0805_2012Metric, symbol Device:R
- C19, C27, C29, C30: footprint Capacitor_SMD:C_0805_2012Metric -> Capacitor_SMD:C_0603_1608Metric
- Q17: value IRLML0100TRPbF -> DMN10H220L-7
- R13: value 220k -> 100k
- R31: value 3.3k -> 22
- R33: value 100k -> 10k
- R62, R63, R65: value 10 -> 22
Connections:
- net at R18.1, U11.3 (IN): now also R23.2; no longer R13.2
- new net: R13.2, R23.1
Other:
- moved on the sheet: R13
Changed lines of the file:
@@
 L Device:R R13
 U 1 1 5B0461F5
-P 700 1300
-F 0 "R13" V 600 1300 50  0000 C CNN
-F 1 "220k" V 700 1300 50  0000 C CNN
-F 2 "Resistor_SMD:R_0805_2012Metric" V 630 1300 50  0001 C CNN
-F 3 "~" H 700 1300 50  0001 C CNN
-	1    700  1300
+P 700 1100
+F 0 "R13" V 600 1100 50  0000 C CNN
+F 1 "100k" V 700 1100 50  0000 C CNN
+F 2 "Resistor_SMD:R_0805_2012Metric" V 630 1100 50  0001 C CNN
+F 3 "~" H 700 1100 50  0001 C CNN
+	1    700  1100
 	1    0    0    -1
 $EndComp
@@
 $EndComp
 Wire Wire Line
-	700  1450 700  1650
-Wire Wire Line
 	700  1650 1600 1650
-Connection ~ 700  1650
 Wire Wire Line
 	700  1650 700  1750
@@
 P 1450 7400
 F 0 "R33" V 1350 7400 50  0000 C CNN
-F 1 "100k" V 1450 7400 50  0000 C CNN
+F 1 "10k" V 1450 7400 50  0000 C CNN
 F 2 "Resistor_SMD:R_0805_2012Metric" V 1380 7400 50  0001 C CNN
 F 3 "~" H 1450 7400 50  0001 C CNN
@@
 P 1200 7250
 F 0 "R31" V 1100 7250 50  0000 C CNN
-F 1 "3.3k" V 1200 7250 50  0000 C CNN
+F 1 "22" V 1200 7250 50  0000 C CNN
 F 2 "Resistor_SMD:R_0805_2012Metric" V 1130 7250 50  0001 C CNN
 F 3 "~" H 1200 7250 50  0001 C CNN
@@
 	4750 7750 4750 6450
 Wire Wire Line
-	700  950  700  1150
-Wire Wire Line
 	1000 950  1000 1150
 Text Label 3200 1300 2    50   ~ 0
@@
 P 1750 7250
 F 0 "Q17" H 1954 7296 50  0000 L CNN
-F 1 "IRLML0100TRPbF" H 1954 7205 50  0000 L CNN
+F 1 "DMN10H220L-7 " H 1954 7205 50  0000 L CNN
 F 2 "Package_TO_SOT_SMD:SOT-23" H 1950 7350 50  0001 C CNN
 F 3 "https://www.mouser.it/datasheet/2/196/irlml0100pbf-1228126.pdf" H 1750 7250 50  0001 C CNN
@@
 F 0 "C19" V 500 3550 50  0000 C CNN
 F 1 "100n" V 800 3550 50  0000 C CNN
-F 2 "Capacitor_SMD:C_0805_2012Metric" H 688 3400 50  0001 C CNN
+F 2 "Capacitor_SMD:C_0603_1608Metric" H 688 3400 50  0001 C CNN
 F 3 "~" H 650 3550 50  0001 C CNN
 	1    650  3550
@@
 F 0 "C27" V 1200 3650 50  0000 C CNN
 F 1 "100n" V 1500 3650 50  0000 C CNN
-F 2 "Capacitor_SMD:C_0805_2012Metric" H 1388 3500 50  0001 C CNN
+F 2 "Capacitor_SMD:C_0603_1608Metric" H 1388 3500 50  0001 C CNN
 F 3 "~" H 1350 3650 50  0001 C CNN
 	1    1350 3650
@@
 F 0 "C29" V 3700 3150 50  0000 C CNN
 F 1 "100n" V 4000 3150 50  0000 C CNN
-F 2 "Capacitor_SMD:C_0805_2012Metric" H 3888 3000 50  0001 C CNN
+F 2 "Capacitor_SMD:C_0603_1608Metric" H 3888 3000 50  0001 C CNN
 F 3 "~" H 3850 3150 50  0001 C CNN
 	1    3850 3150
@@
 P 9300 3500
 F 0 "R65" V 9400 3500 50  0000 C CNN
-F 1 "10" V 9300 3500 50  0000 C CNN
+F 1 "22" V 9300 3500 50  0000 C CNN
 F 2 "Resistor_SMD:R_0805_2012Metric" V 9230 3500 50  0001 C CNN
 F 3 "~" H 9300 3500 50  0001 C CNN
@@
 Wire Notes Line
 	2300 6150 2300 4650
-Text Notes 9550 2250 0    50   ~ 0
+Text Notes 10100 2350 0    50   ~ 0
 Actual daisychain connection \nof the shutdown line
 $Comp
@@
 F 0 "C30" V 7900 2750 50  0000 C CNN
 F 1 "100n" V 8200 2750 50  0000 C CNN
-F 2 "Capacitor_SMD:C_0805_2012Metric" H 8088 2600 50  0001 C CNN
+F 2 "Capacitor_SMD:C_0603_1608Metric" H 8088 2600 50  0001 C CNN
 F 3 "~" H 8050 2750 50  0001 C CNN
 	1    8050 2750
@@
 $EndComp
 $Comp
-L Device:Q_NMOS_GSD Q18
-U 1 1 60521BAF
-P 5700 4850
-F 0 "Q18" H 5900 4900 50  0000 L CNN
-F 1 "TSM2306" H 5900 4800 50  0000 L CNN
-F 2 "Package_TO_SOT_SMD:SOT-23" H 5900 4950 50  0001 C CNN
-F 3 "http://www.taiwansemi.com/products/datasheet/TSM2306_B15.pdf" H 5700 4850 50  0001 C CNN
-	1    5700 4850
-	1    0    0    -1
-$EndComp
-$Comp
 L Device:R R62
 U 1 1 60555676
 P 5500 4700
 F 0 "R62" V 5600 4700 50  0000 C CNN
-F 1 "10" V 5500 4700 50  0000 C CNN
+F 1 "22" V 5500 4700 50  0000 C CNN
 F 2 "Resistor_SMD:R_0805_2012Metric" V 5430 4700 50  0001 C CNN
 F 3 "~" H 5500 4700 50  0001 C CNN
@@
 P 6400 4750
 F 0 "R63" V 6500 4750 50  0000 C CNN
-F 1 "10" V 6400 4750 50  0000 C CNN
+F 1 "22" V 6400 4750 50  0000 C CNN
 F 2 "Resistor_SMD:R_0805_2012Metric" V 6330 4750 50  0001 C CNN
 F 3 "~" H 6400 4750 50  0001 C CNN
@@
 Wire Wire Line
 	6550 7000 6850 7000
+$Comp
+L Device:Q_NMOS_GSD Q18
+U 1 1 60521BAF
+P 5700 4850
+F 0 "Q18" H 5900 4900 50  0000 L CNN
+F 1 "TSM2306" H 5900 4800 50  0000 L CNN
+F 2 "Package_TO_SOT_SMD:SOT-23" H 5900 4950 50  0001 C CNN
+F 3 "http://www.taiwansemi.com/products/datasheet/TSM2306_B15.pdf" H 5700 4850 50  0001 C CNN
+	1    5700 4850
+	1    0    0    -1
+$EndComp
+$Comp
+L Device:R R23
+U 1 1 60DE7370
+P 700 1400
+F 0 "R23" V 600 1400 50  0000 C CNN
+F 1 "100k" V 700 1400 50  0000 C CNN
+F 2 "Resistor_SMD:R_0805_2012Metric" V 630 1400 50  0001 C CNN
+F 3 "~" H 700 1400 50  0001 C CNN
+	1    700  1400
+	1    0    0    -1
+$EndComp
+Wire Wire Line
+	700  1550 700  1650
+Connection ~ 700  1650
 $EndSCHEMATC
