File: mainboard/HVSide.sch (KiCad schematic (older format))
At the start: 51 parts, among them J10 IMD_TS-, J7 ProminentIndicator, J8 HV, J9 IMD_TS+, Q15 BULB49D, Q16 NTR4003, U14 Si8901, U15 LTC6259, U17 REF2940, U18 FODM611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

Commit message: finished footprint association
Parts:
- C13: footprint (none) -> Capacitor_SMD:C_0805_2012Metric
- C31, C32: value 10u -> 4.7u; footprint (none) -> Capacitor_SMD:C_0805_2012Metric
- C33, C34: renamed from C?; value 1uF -> 1u; footprint (none) -> Capacitor_SMD:C_0805_2012Metric
- Q16: value NTR4003 -> TSM2306
- R36, R37: value 390K -> 390k
- R47: value 100K -> 100k
- R54, R55, R56, R59: footprint (none) -> Resistor_SMD:R_0805_2012Metric
- U14: footprint (none) -> Package_SO:SOIC-16W_7.5x10.3mm_P1.27mm
- U22: footprint (none) -> Package_TO_SOT_SMD:SOT-223-3_TabPin2
- U23: footprint (none) -> MainBoard:RFMM-0505S
- U24: renamed from U?; footprint (none) -> MainBoard:ROE-0505S
- gave numbers to parts that had none: 5
- renumbered D5 to DZ5, D6 to DZ6, D7 to DZ7
Changed lines of the file:
@@
 	1750 2250 1750 2350
 $Comp
-L Device:D_Zener D6
+L Device:D_Zener DZ6
 U 1 1 5B50F5FB
 P 1350 2000
-F 0 "D6" H 1350 1900 50  0000 C CNN
+F 0 "DZ6" H 1350 1900 50  0000 C CNN
 F 1 "MMBZ4624 4V7" H 1350 2100 50  0000 C CNN
 F 2 "Diode_SMD:D_SOT-23_ANK" H 1350 2000 50  0001 C CNN
@@
 	1350 1650 1350 1850
 $Comp
-L Device:D_Zener D5
+L Device:D_Zener DZ5
 U 1 1 5B50F604
 P 1700 750
-F 0 "D5" H 1700 650 50  0000 C CNN
+F 0 "DZ5" H 1700 650 50  0000 C CNN
 F 1 "BZD27C56P 56V" H 1700 850 50  0000 C CNN
 F 2 "MainBoard:DO-219AB" H 1700 750 50  0001 C CNN
@@
 P 1050 1200
 F 0 "R36" V 950 1200 50  0000 C CNN
-F 1 "390K" V 1050 1200 50  0000 C CNN
+F 1 "390k" V 1050 1200 50  0000 C CNN
 F 2 "Resistor_SMD:R_2512_6332Metric" V 980 1200 50  0001 C CNN
 F 3 "~" H 1050 1200 50  0001 C CNN
@@
 P 1350 1200
 F 0 "R37" V 1250 1200 50  0000 C CNN
-F 1 "390K" V 1350 1200 50  0000 C CNN
+F 1 "390k" V 1350 1200 50  0000 C CNN
 F 2 "Resistor_SMD:R_2512_6332Metric" V 1280 1200 50  0001 C CNN
 F 3 "~" H 1350 1200 50  0001 C CNN
@@
 P 4900 6750
 F 0 "R47" V 4800 6750 50  0000 C CNN
-F 1 "100K" V 4900 6750 50  0000 C CNN
+F 1 "100k" V 4900 6750 50  0000 C CNN
 F 2 "Resistor_SMD:R_0805_2012Metric" V 4830 6750 50  0001 C CNN
 F 3 "~" H 4900 6750 50  0001 C CNN
@@
 	5300 6300 5300 6200
 $Comp
-L Device:D_Zener D7
+L Device:D_Zener DZ7
 U 1 1 5B28B6F4
 P 2050 1000
-F 0 "D7" H 2050 900 50  0000 C CNN
+F 0 "DZ7" H 2050 900 50  0000 C CNN
 F 1 "MMBZ4624 4V7" H 2050 1100 50  0000 C CNN
 F 2 "Diode_SMD:D_SOT-23_ANK" H 2050 1000 50  0001 C CNN
@@
 F 0 "C13" H 6142 1046 50  0000 L CNN
 F 1 "10n" H 6142 955 50  0000 L CNN
-F 2 "" H 6050 1000 50  0001 C CNN
+F 2 "Capacitor_SMD:C_0805_2012Metric" H 6050 1000 50  0001 C CNN
 F 3 "~" H 6050 1000 50  0001 C CNN
 	1    6050 1000
@@
 F 0 "R54" H 6409 1046 50  0000 L CNN
 F 1 "2k" H 6409 955 50  0000 L CNN
-F 2 "" H 6350 1000 50  0001 C CNN
+F 2 "Resistor_SMD:R_0805_2012Metric" H 6350 1000 50  0001 C CNN
 F 3 "~" H 6350 1000 50  0001 C CNN
 	1    6350 1000
@@
 F 0 "R55" H 6809 1296 50  0000 L CNN
 F 1 "680" H 6809 1205 50  0000 L CNN
-F 2 "" H 6750 1250 50  0001 C CNN
+F 2 "Resistor_SMD:R_0805_2012Metric" H 6750 1250 50  0001 C CNN
 F 3 "~" H 6750 1250 50  0001 C CNN
 	1    6750 1250
@@
 F 0 "R56" H 6809 1596 50  0000 L CNN
 F 1 "100k" H 6809 1505 50  0000 L CNN
-F 2 "" H 6750 1550 50  0001 C CNN
+F 2 "Resistor_SMD:R_0805_2012Metric" H 6750 1550 50  0001 C CNN
 F 3 "~" H 6750 1550 50  0001 C CNN
 	1    6750 1550
@@
 F 0 "U14" H 4700 1875 50  0000 C CNN
 F 1 "Si8901" H 4700 1784 50  0000 C CNN
-F 2 "" H 4550 1800 50  0001 C CNN
+F 2 "Package_SO:SOIC-16W_7.5x10.3mm_P1.27mm" H 4550 1800 50  0001 C CNN
 F 3 "" H 4550 1800 50  0001 C CNN
 	1    4700 1350
@@
 F 0 "R59" V 4200 1850 50  0000 C CNN
 F 1 "5k" V 4150 1650 50  0000 C CNN
-F 2 "" V 4080 1650 50  0001 C CNN
+F 2 "Resistor_SMD:R_0805_2012Metric" V 4080 1650 50  0001 C CNN
 F 3 "~" H 4150 1650 50  0001 C CNN
 	1    4150 1650
@@
 F 0 "U22" H 8550 2692 50  0000 C CNN
 F 1 "LM1117-3.3" H 8550 2601 50  0000 C CNN
-F 2 "" H 8550 2450 50  0001 C CNN
+F 2 "Package_TO_SOT_SMD:SOT-223-3_TabPin2" H 8550 2450 50  0001 C CNN
 F 3 "http://www.ti.com/lit/ds/symlink/lm1117.pdf" H 8550 2450 50  0001 C CNN
 	1    8550 2450
@@
 P 9250 2600
 F 0 "C32" H 9365 2646 50  0000 L CNN
-F 1 "10u" H 9365 2555 50  0000 L CNN
-F 2 "" H 9288 2450 50  0001 C CNN
+F 1 "4.7u" H 9365 2555 50  0000 L CNN
+F 2 "Capacitor_SMD:C_0805_2012Metric" H 9288 2450 50  0001 C CNN
 F 3 "~" H 9250 2600 50  0001 C CNN
 	1    9250 2600
@@
 F 0 "U23" H 9050 1475 50  0000 C CNN
 F 1 "RFMM-0505S" H 9050 1384 50  0000 C CNN
-F 2 "" H 8750 1250 50  0001 C CNN
+F 2 "MainBoard:RFMM-0505S" H 8750 1250 50  0001 C CNN
 F 3 "" H 8750 1250 50  0001 C CNN
 	1    8750 1250
@@
 P 7950 1350
 F 0 "C31" H 8065 1396 50  0000 L CNN
-F 1 "10u" H 8065 1305 50  0000 L CNN
-F 2 "" H 7988 1200 50  0001 C CNN
+F 1 "4.7u" H 8065 1305 50  0000 L CNN
+F 2 "Capacitor_SMD:C_0805_2012Metric" H 7988 1200 50  0001 C CNN
 F 3 "~" H 7950 1350 50  0001 C CNN
 	1    7950 1350
@@
 AR Path="/5B50ED38/6066CB94" Ref="Q16"  Part="1"
 F 0 "Q16" H 5400 6550 50  0000 L CNN
-F 1 "NTR4003" H 5400 6450 50  0000 L CNN
+F 1 "TSM2306" H 5400 6450 50  0000 L CNN
 F 2 "Package_TO_SOT_SMD:SOT-23" H 5400 6600 50  0001 C CNN
 F 3 "http://www.taiwansemi.com/products/datasheet/TSM2306_B15.pdf" H 5200 6500 50  0001 C CNN
@@
 $EndComp
 $Comp
-L MainBoard:ROE-0505S U?
+L MainBoard:ROE-0505S U24
 U 1 1 6063CC87
 P 2850 2850
-F 0 "U?" H 3150 3075 50  0000 C CNN
+F 0 "U24" H 3150 3075 50  0000 C CNN
 F 1 "ROE-0505S" H 3150 2984 50  0000 C CNN
-F 2 "" H 2850 2850 50  0001 C CNN
+F 2 "MainBoard:ROE-0505S" H 2850 2850 50  0001 C CNN
 F 3 "" H 2850 2850 50  0001 C CNN
 	1    2850 2850
@@
 $EndComp
 $Comp
-L Connector_Generic:Conn_02x02_Odd_Even J?
+L Connector_Generic:Conn_02x02_Odd_Even J12
 U 1 1 6066BC41
 P 1350 2900
-F 0 "J?" H 1400 3117 50  0000 C CNN
+F 0 "J12" H 1400 3117 50  0000 C CNN
 F 1 "PROMINENT" H 1400 3026 50  0000 C CNN
 F 2 "Connector_Molex:Molex_Micro-Fit_3.0_43045-0412_2x02_P3.00mm_Vertical" H 1350 2900 50  0001 C CNN
@@
 	1650 2900 2150 2900
 $Comp
-L Comparator:ADCMP350 U?
+L Comparator:ADCMP350 U12
 U 1 1 6069F7D8
 P 1450 3650
-F 0 "U?" H 1600 3400 50  0000 L CNN
+F 0 "U12" H 1600 3400 50  0000 L CNN
 F 1 "ADCMP350" H 1600 3500 50  0000 L CNN
 F 2 "Package_TO_SOT_SMD:Analog_KS-4" H 1450 3250 50  0001 C CNN
@@
 $EndComp
 $Comp
-L Device:C C?
+L Device:C C33
 U 1 1 606CADF0
 P 2450 2900
-F 0 "C?" H 2565 2946 50  0000 L CNN
-F 1 "1uF" H 2565 2855 50  0000 L CNN
-F 2 "" H 2488 2750 50  0001 C CNN
+F 0 "C33" H 2565 2946 50  0000 L CNN
+F 1 "1u" H 2565 2855 50  0000 L CNN
+F 2 "Capacitor_SMD:C_0805_2012Metric" H 2488 2750 50  0001 C CNN
 F 3 "~" H 2450 2900 50  0001 C CNN
 	1    2450 2900
@@
 $EndComp
 $Comp
-L Device:C C?
+L Device:C C34
 U 1 1 606CBC1F
 P 3800 2950
-F 0 "C?" H 3915 2996 50  0000 L CNN
-F 1 "1uF" H 3915 2905 50  0000 L CNN
-F 2 "" H 3838 2800 50  0001 C CNN
+F 0 "C34" H 3915 2996 50  0000 L CNN
+F 1 "1u" H 3915 2905 50  0000 L CNN
+F 2 "Capacitor_SMD:C_0805_2012Metric" H 3838 2800 50  0001 C CNN
 F 3 "~" H 3800 2950 50  0001 C CNN
 	1    3800 2950
@@
 	1450 3300 1450 3350
 $Comp
-L Device:R R?
+L Device:R R17
 U 1 1 6074A3F8
 P 1650 3300
-F 0 "R?" V 1550 3300 50  0000 C CNN
+F 0 "R17" V 1550 3300 50  0000 C CNN
 F 1 "1k" V 1650 3300 50  0000 C CNN
 F 2 "Resistor_SMD:R_0805_2012Metric" V 1580 3300 50  0001 C CNN
@@
 	6100 3000 6350 3000
 $Comp
-L power:-BATT #PWR?
+L power:-BATT #PWR068
 U 1 1 607C6E3B
 P 1450 4050
-F 0 "#PWR?" H 1450 3900 50  0001 C CNN
+F 0 "#PWR068" H 1450 3900 50  0001 C CNN
 F 1 "-BATT" H 1450 4200 50  0000 C CNN
 F 2 "" H 1450 4050 50  0001 C CNN
@@
 $EndComp
 $Comp
-L power:-BATT #PWR?
+L power:-BATT #PWR073
 U 1 1 607D0B9A
 P 3650 3150
-F 0 "#PWR?" H 3650 3000 50  0001 C CNN
+F 0 "#PWR073" H 3650 3000 50  0001 C CNN
 F 1 "-BATT" H 3650 3300 50  0000 C CNN
 F 2 "" H 3650 3150 50  0001 C CNN
@@
 $EndComp
 $Comp
-L Device:R R?
+L Device:R R12
 U 1 1 608059E6
 P 1000 3650
-F 0 "R?" V 900 3650 50  0000 C CNN
+F 0 "R12" V 900 3650 50  0000 C CNN
 F 1 "10M" V 1000 3650 50  0000 C CNN
 F 2 "Resistor_SMD:R_1210_3225Metric" V 930 3650 50  0001 C CNN
@@
 $EndComp
 $Comp
-L Device:R R?
+L Device:R R16
 U 1 1 60805E48
 P 1200 3850
-F 0 "R?" V 1100 3850 50  0000 C CNN
+F 0 "R16" V 1100 3850 50  0000 C CNN
 F 1 "100k" V 1200 3850 50  0000 C CNN
 F 2 "Resistor_SMD:R_0805_2012Metric" V 1130 3850 50  0001 C CNN
@@
 	1200 3650 1250 3650
 $Comp
-L MainBoard:+TS #PWR?
+L MainBoard:+TS #PWR065
 U 1 1 6088B923
 P 750 3650
-F 0 "#PWR?" H 750 3500 50  0001 C CNN
+F 0 "#PWR065" H 750 3500 50  0001 C CNN
 F 1 "+TS" V 650 3650 50  0000 L CNN
 F 2 "" H 650 3400 50  0001 C CNN

Commit message: Done early board
Parts:
- removed DZ5: BZD27C56P 56V, MainBoard:DO-219AB, symbol Device:D_Zener
- removed DZ6, DZ7: MMBZ4624 4V7, Diode_SMD:D_SOT-23_ANK, symbol Device:D_Zener
- removed F1: 0885001.DR, MainBoard:SMD_Fuse, symbol Device:Fuse
- removed J7: ProminentIndicator, Connector_Molex:Molex_Micro-Fit_3.0_43650-0215_1x02_P3.00mm_Vertical, symbol Connector_Generic:Conn_01x02
- removed Q15: BULB49D, MainBoard:D2PAK, symbol Device:Q_NPN_BCE
- removed R36, R37: 390k, Resistor_SMD:R_2512_6332Metric, symbol Device:R
- removed R38: 330, Resistor_SMD:R_0805_2012Metric, symbol Device:R
Other:
- note removed: "4.7V in the connector \nwhen V_TS>60V"
- note removed: "CRCW2512"
- note removed: "Limited at 4.7V by D7\nC503B High Brightness LED"
- note removed: "V_TS max is 600V"
- note removed: "old PROMINENT INDICATOR CURRENT SOURCE"
- moved on the sheet: C13, C25, C26, C28, C31, C32, C33, C34, J12, R12, R16, R17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

Commit message: board soldered
Parts:
- removed U14: Si8901, Package_SO:SOIC-16W_7.5x10.3mm_P1.27mm, symbol si8900:Si8901
- removed U17: REF2940, Package_TO_SOT_SMD:SOT-23, symbol MainBoard:REF2940
- added C6: 100n, Capacitor_SMD:C_0603_1608Metric, symbol Device:C
- added R19, R21: 22, Resistor_SMD:R_0805_2012Metric, symbol Device:R_Small
- added R24: 1k, Resistor_SMD:R_0805_2012Metric, symbol Device:R_Small
- added U3: Si8900, MainBoard:SOIC-16, symbol si8900:Si8900
- C13, C26, C28: footprint Capacitor_SMD:C_0805_2012Metric -> Capacitor_SMD:C_0603_1608Metric
- R54: value 2k -> 1k
- R55: value 680 -> 1k
- R59: value 5k -> 1k
- U15: footprint MainBoard:MSOP-8 -> MainBoard:MSOP-8_and_TSOT-23-8
Connections:
- net 4VISO is gone; now on net 5VISO: C28.1, U15.8, U15.8
- net +3V3: now also U3.10 (VDDB), U3.16 (VDDB)
- net -BATT: now also C6.2, U3.8 (GNDA)
- net 3V3ISO: now also C6.1, R24.2, U3.1 (VDDA); no longer R54.1
- net GND: now also U3.9 (GNDB)
- net PackV: now also U3.4 (AIN1)
- net TSV: now also U3.3 (AIN0)
- net ~RST~_ADCA: now also R54.1, U3.6 (NC); no longer R54.2
- net at R59.2: now also U3.7 (~RST)
- new net: R24.1, R54.2
- new net: R21.2, U3.12 (TX)
- new net: R19.1, U3.13 (RX)
- new net ADC_RX: R19.2
- new net ADC_TX: R21.1
Other:
- note added: "LTC6259 can be replaced by a LM358?"
- note removed: "25mA max"
- note removed: "ISOLATED 4V VOLTAGE REFERENCE"
- moved on the sheet: C28, R54
Changed lines of the file:
@@
 F 0 "U15" H 6000 1350 50  0000 L CNN
 F 1 "LTC6259" H 6000 1050 50  0000 L CNN
-F 2 "MainBoard:MSOP-8" H 6000 950 50  0001 L CNN
+F 2 "MainBoard:MSOP-8_and_TSOT-23-8" H 6000 950 50  0001 L CNN
 F 3 "www.analog.com/media/en/technical-documentation/data-sheets/6258960fa.pdf" H 5950 1150 50  0001 C CNN
 	1    5950 1200
@@
 F 0 "U15" H 6000 2550 50  0000 L CNN
 F 1 "LTC6259" H 6000 2250 50  0000 L CNN
-F 2 "MainBoard:MSOP-8" H 6000 2150 50  0001 L CNN
+F 2 "MainBoard:MSOP-8_and_TSOT-23-8" H 6000 2150 50  0001 L CNN
 F 3 "www.analog.com/media/en/technical-documentation/data-sheets/6258960fa.pdf" H 5950 2350 50  0001 C CNN
 	2    5950 2400
@@
 F 0 "C26" V 10350 3500 50  0000 C CNN
 F 1 "100n" V 10650 3500 50  0000 C CNN
-F 2 "Capacitor_SMD:C_0805_2012Metric" H 10538 3350 50  0001 C CNN
+F 2 "Capacitor_SMD:C_0603_1608Metric" H 10538 3350 50  0001 C CNN
 F 3 "~" H 10500 3500 50  0001 C CNN
 	1    10500 3500
@@
 Wire Wire Line
 	5900 1900 5900 2100
-Text Label 5900 700  3    50   ~ 0
-4VISO
-Text Label 5900 1900 3    50   ~ 0
-4VISO
-$Comp
-L MainBoard:REF2940 U17
-U 1 1 5B56F9B4
-P 8550 5700
-F 0 "U17" H 8550 6015 50  0000 C CNN
-F 1 "REF2940" H 8550 5924 50  0000 C CNN
-F 2 "Package_TO_SOT_SMD:SOT-23" H 8550 5500 50  0001 C CNN
-F 3 "www.ti.com/lit/ds/symlink/ref2940.pdf" H 8550 5700 50  0001 C CNN
-	1    8550 5700
-	1    0    0    -1
-$EndComp
-Wire Wire Line
-	8250 5650 8050 5650
-Text Label 8050 5650 0    50   ~ 0
-5VISO
-Wire Wire Line
-	8250 5750 8150 5750
-$Comp
-L power:-BATT #PWR0129
-U 1 1 5B56F9BE
-P 8150 5750
-F 0 "#PWR0129" H 8150 5600 50  0001 C CNN
-F 1 "-BATT" V 8150 5900 50  0000 L CNN
-F 2 "" H 8150 5750 50  0001 C CNN
-F 3 "" H 8150 5750 50  0001 C CNN
-	1    8150 5750
-	0    -1   -1   0
-$EndComp
-Wire Wire Line
-	8850 5650 9050 5650
-Text Label 9050 5650 2    50   ~ 0
-4VISO
-Wire Wire Line
-	9050 5650 9050 5750
 $Comp
 L Device:C C28
 U 1 1 5B56F9C7
-P 9050 5900
-F 0 "C28" V 8900 5900 50  0000 C CNN
-F 1 "100n" V 9200 5900 50  0000 C CNN
-F 2 "Capacitor_SMD:C_0805_2012Metric" H 9088 5750 50  0001 C CNN
-F 3 "~" H 9050 5900 50  0001 C CNN
-	1    9050 5900
-	1    0    0    -1
-$EndComp
-Wire Wire Line
-	9050 6050 9050 6150
+P 4550 1750
+F 0 "C28" V 4400 1750 50  0000 C CNN
+F 1 "100n" V 4700 1750 50  0000 C CNN
+F 2 "Capacitor_SMD:C_0603_1608Metric" H 4588 1600 50  0001 C CNN
+F 3 "~" H 4550 1750 50  0001 C CNN
+	1    4550 1750
+	1    0    0    -1
+$EndComp
+Wire Wire Line
+	4550 1900 4550 2000
 $Comp
 L power:-BATT #PWR0131
 U 1 1 5B56F9CF
-P 9050 6150
-F 0 "#PWR0131" H 9050 6000 50  0001 C CNN
-F 1 "-BATT" H 9050 6300 50  0000 C CNN
-F 2 "" H 9050 6150 50  0001 C CNN
-F 3 "" H 9050 6150 50  0001 C CNN
-	1    9050 6150
+P 4550 2000
+F 0 "#PWR0131" H 4550 1850 50  0001 C CNN
+F 1 "-BATT" H 4550 2150 50  0000 C CNN
+F 2 "" H 4550 2000 50  0001 C CNN
+F 3 "" H 4550 2000 50  0001 C CNN
+	1    4550 2000
 	-1   0    0    1
 $EndComp
@@
 ISOLATED 5V VOLTAGE SOURCE
 Wire Notes Line
-	9300 5300 9300 6400
-Wire Notes Line
-	9300 6400 7700 6400
-Wire Notes Line
-	7700 6400 7700 5300
-Wire Notes Line
-	7700 5300 9300 5300
-Text Notes 7700 5300 0    50   ~ 0
-ISOLATED 4V VOLTAGE REFERENCE
-Wire Notes Line
 	7700 4100 7700 5200
 Wire Notes Line
@@
 Wire Wire Line
 	8850 1300 8800 1300
-Text HLabel 8850 1300 2    50   Input ~ 0
-SDA
-Text HLabel 8850 1200 2    50   Input ~ 0
-SCL
 Text Label 7600 1400 0    50   ~ 0
 ~RST~_ADCA
@@
 F 0 "C13" H 9842 896 50  0000 L CNN
 F 1 "10n" H 9842 805 50  0000 L CNN
-F 2 "Capacitor_SMD:C_0805_2012Metric" H 9750 850 50  0001 C CNN
+F 2 "Capacitor_SMD:C_0603_1608Metric" H 9750 850 50  0001 C CNN
 F 3 "~" H 9750 850 50  0001 C CNN
 	1    9750 850
@@
 L Device:R_Small R54
 U 1 1 60507EA6
-P 10050 850
-F 0 "R54" H 10109 896 50  0000 L CNN
-F 1 "2k" H 10109 805 50  0000 L CNN
-F 2 "Resistor_SMD:R_0805_2012Metric" H 10050 850 50  0001 C CNN
-F 3 "~" H 10050 850 50  0001 C CNN
-	1    10050 850
-	1    0    0    -1
+P 10350 700
+F 0 "R54" V 10450 650 50  0000 L CNN
+F 1 "1k" V 10350 650 50  0000 L CNN
+F 2 "Resistor_SMD:R_0805_2012Metric" H 10350 700 50  0001 C CNN
+F 3 "~" H 10350 700 50  0001 C CNN
+	1    10350 700
+	0    1    1    0
 $EndComp
 Wire Wire Line
 	9450 700  9750 700
-Wire Wire Line
-	10050 700  10050 750
 Wire Wire Line
 	9750 750  9750 700
@@
 Wire Wire Line
 	9750 700  10050 700
-Wire Wire Line
-	10050 950  10050 1000
-Wire Wire Line
-	10050 1000 9750 1000
 Wire Wire Line
 	9750 950  9750 1000
@@
 P 10450 1100
 F 0 "R55" H 10509 1146 50  0000 L CNN
-F 1 "680" H 10509 1055 50  0000 L CNN
+F 1 "1k" H 10509 1055 50  0000 L CNN
 F 2 "Resistor_SMD:R_0805_2012Metric" H 10450 1100 50  0001 C CNN
 F 3 "~" H 10450 1100 50  0001 C CNN
@@
 	8000 1100 7700 1100
 $Comp
-L si8900:Si8901 U14
-U 1 1 603E5D4E
-P 8400 1200
-F 0 "U14" H 8400 1725 50  0000 C CNN
-F 1 "Si8901" H 8400 1634 50  0000 C CNN
-F 2 "Package_SO:SOIC-16W_7.5x10.3mm_P1.27mm" H 8250 1650 50  0001 C CNN
-F 3 "" H 8250 1650 50  0001 C CNN
-	1    8400 1200
-	1    0    0    -1
-$EndComp
-$Comp
 L Device:R R59
 U 1 1 603F9D47
 P 7850 1500
 F 0 "R59" V 7900 1700 50  0000 C CNN
-F 1 "5k" V 7850 1500 50  0000 C CNN
+F 1 "1k" V 7850 1500 50  0000 C CNN
 F 2 "Resistor_SMD:R_0805_2012Metric" V 7780 1500 50  0001 C CNN
 F 3 "~" H 7850 1500 50  0001 C CNN
@@
 Text Label 7700 900  0    50   ~ 0
 3V3ISO
-Text Notes 8800 5550 0    50   ~ 0
-25mA max
 $Comp
 L Device:Q_NMOS_GSD Q?
@@
 Text Notes 700  1750 0    50   ~ 0
 CRMA1210
+$Comp
+L si8900:Si8900 U3
+U 1 1 60A92D55
+P 8400 1200
+F 0 "U3" H 8400 1725 50  0000 C CNN
+F 1 "Si8900" H 8400 1634 50  0000 C CNN
+F 2 "MainBoard:SOIC-16" H 8250 1650 50  0001 C CNN
+F 3 "" H 8250 1650 50  0001 C CNN
+	1    8400 1200
+	1    0    0    -1
+$EndComp
+$Comp
+L Device:R_Small R19
+U 1 1 60AA86E5
+P 8950 1200
+F 0 "R19" V 9000 1200 50  0000 C CNN
+F 1 "22" V 8950 1150 50  0000 L CNN
+F 2 "Resistor_SMD:R_0805_2012Metric" H 8950 1200 50  0001 C CNN
+F 3 "~" H 8950 1200 50  0001 C CNN
+	1    8950 1200
+	0    -1   -1   0
+$EndComp
+$Comp
+L Device:R_Small R21
+U 1 1 60AA8C19
+P 8950 1300
+F 0 "R21" V 9000 1300 50  0000 C CNN
+F 1 "22" V 8950 1250 50  0000 L CNN
+F 2 "Resistor_SMD:R_0805_2012Metric" H 8950 1300 50  0001 C CNN
+F 3 "~" H 8950 1300 50  0001 C CNN
+	1    8950 1300
+	0    1    1    0
+$EndComp
+Text HLabel 9100 1200 2    50   Input ~ 0
+ADC_RX
+Text HLabel 9100 1300 2    50   Output ~ 0
+ADC_TX
+Wire Wire Line
+	9050 1200 9100 1200
+Wire Wire Line
+	9100 1300 9050 1300
+Text Label 5900 700  3    50   ~ 0
+5VISO
+Text Label 5900 1900 3    50   ~ 0
+5VISO
+Text Label 4550 1350 3    50   ~ 0
+5VISO
+Wire Wire Line
+	4550 1600 4550 1350
+$Comp
+L Device:C C6
+U 1 1 60B31754
+P 7350 900
+F 0 "C6" V 7200 900 50  0000 C CNN
+F 1 "100n" V 7500 900 50  0000 C CNN
+F 2 "Capacitor_SMD:C_0603_1608Metric" H 7388 750 50  0001 C CNN
+F 3 "~" H 7350 900 50  0001 C CNN
+	1    7350 900
+	1    0    0    -1
+$EndComp
+Wire Wire Line
+	7350 1050 7350 1150
+$Comp
+L power:-BATT #PWR0147
+U 1 1 60B3175B
+P 7350 1150
+F 0 "#PWR0147" H 7350 1000 50  0001 C CNN
+F 1 "-BATT" H 7350 1300 50  0000 C CNN
+F 2 "" H 7350 1150 50  0001 C CNN
+F 3 "" H 7350 1150 50  0001 C CNN
+	1    7350 1150
+	-1   0    0    1
+$EndComp
+Wire Wire Line
+	7700 900  7700 750
+Wire Wire Line
+	7700 750  7350 750
+$Comp
+L Device:R_Small R24
+U 1 1 60DF6006
+P 10150 700
+F 0 "R24" V 10250 650 50  0000 L CNN
+F 1 "1k" V 10150 650 50  0000 L CNN
+F 2 "Resistor_SMD:R_0805_2012Metric" H 10150 700 50  0001 C CNN
+F 3 "~" H 10150 700 50  0001 C CNN
+	1    10150 700
+	0    1    1    0
+$EndComp
+Wire Wire Line
+	10200 1000 10200 900
+Wire Wire Line
+	10200 900  10500 900
+Wire Wire Line
+	10500 900  10500 700
+Wire Wire Line
+	10500 700  10450 700
+Wire Wire Line
+	9750 1000 10200 1000
+Text Notes 4350 3200 0    50   ~ 0
+LTC6259 can be replaced by a LM358?
 $EndSCHEMATC
