File: mainboard/MainBoard.kicad_pcb (KiCad board)
At the start: 4 copper layers, 365 x 60 mm, 136 parts, among them J1 isoSPI, J10 IMD_TS-, J2 SWDebug, J3 IMD, J4 IO, J5 AIR-, J6 AIR+, J7 ProminentIndicator, J8 HV, J9 IMD_TS+, K1 KT12-1A, Q1 TSM2306, Q10 TSM3401, Q11 TSM3401, Q12 TSM2306, Q13 TSM2312, Q14 BC846AW, Q15 BULB49D, Q16 TSM2312, Q2 TSM3401, Q3 TSM3401, Q4 TSM3401, Q5 TSM2306, Q6 TSM2306, Q7 TSM3401, Q8 TSM2312, Q9 TSM3401, U1 LTC6820, U10 REF2920, U11 MAX16053, U12 SN74LVC1G123, U13 ISOW7841, U14 LTC1865L, U15 LTC6259, U16 REF3433, U17 REF2940, U18 FODM611, U19 TPS3700, U2 HM2103, U3 M24M02, U4 M24M02, U5 STM32F334K8, U6 MicroSD, U7 MCP2562, U8 LP2989, U9 HTFS200-P

Commit message: Done early board
Parts:
- removed C24: 10n, Capacitor_SMD:C_0805_2012Metric
- removed D1, D3: BT150S-600R, MainBoard:TO-252-2
- removed D4, D6, D7: MMBZ4624, Diode_SMD:D_SOT-23_ANK
- removed D5: BZD27C56P, MainBoard:DO-219AB
- removed F1: 0885001.DR, MainBoard:SMD_Fuse
- removed Q10, Q11, Q2, Q3, Q4, Q7, Q9: TSM3401, Package_TO_SOT_SMD:SOT-23
- removed Q12, Q5, Q6: TSM2306, Package_TO_SOT_SMD:SOT-23
- removed Q13, Q8: TSM2312, Package_TO_SOT_SMD:SOT-23
- removed Q15: BULB49D, MainBoard:D2PAK
- removed R21, R22, R27, R29: 100K, Resistor_SMD:R_0805_2012Metric
- removed R23: 1M, Resistor_SMD:R_0805_2012Metric
- removed R24, R25, R28: 10K, Resistor_SMD:R_0805_2012Metric
- removed R26: 3.3K, Resistor_SMD:R_0805_2012Metric
- removed R34, R35: 10K, MainBoard:TO-247_wHeatsink
- removed R36, R37: 390K, Resistor_SMD:R_2512_6332Metric
- removed R38: 330, Resistor_SMD:R_0805_2012Metric
- added C13: 10n, Capacitor_SMD:C_0805_2012Metric, F.Cu at (247.8, 115.3)
- added C19: 100n, Capacitor_SMD:C_0805_2012Metric, B.Cu at (165.8, 114.5)
- added C29: 100n, Capacitor_SMD:C_0805_2012Metric, B.Cu at (157.8, 107.2)
- added C30: 100n, Capacitor_SMD:C_0805_2012Metric, B.Cu at (157.8, 114.5)
- added C31: 4.7u, Capacitor_SMD:C_0805_2012Metric, B.Cu at (224.2, 135.2)
- added C32: 4.7u, Capacitor_SMD:C_0805_2012Metric, F.Cu at (249.8, 135.4)
- added C33: 1u, Capacitor_SMD:C_0805_2012Metric, F.Cu at (300.5, 138.6)
- added C34: 1u, Capacitor_SMD:C_0805_2012Metric, F.Cu at (300.5, 133.3)
- added D8: BAS16GW, Diode_SMD:D_SOD-123, F.Cu at (147.6, 116.3)
- added DZ3: MMBZ4624 4V7, Diode_SMD:D_SOT-23_ANK, F.Cu at (157.5, 92.0)
- added DZ4: MMBZ4624 4V7, Diode_SMD:D_SOT-23_ANK, F.Cu at (127.5, 112.2)
- added G***: LOGO, MainBoard:LOGO, F.Cu at (155.2, 126.7)
- added G***: LOGO, MainBoard:logo_fox, F.Cu at (201.6, 141.8)
- added J11: ON_HANDCART, Connector_PinHeader_2.54mm:PinHeader_1x02_P2.54mm_Vertical, F.Cu at (189.2, 93.7)
- added J12: PROMINENT, Connector_Molex:Molex_Micro-Fit_3.0_43045-0412_2x02_P3.00mm_Vertical, F.Cu at (304.8, 138.1)
- added K2: UMS05-1A80-75L, MainBoard:G6DN-1A_DC12, F.Cu at (147.2, 108.5)
- added Q17: IRLML0100TRPbF, Package_TO_SOT_SMD:SOT-23, F.Cu at (127.5, 116.0)
- added Q18: TSM2306, Package_TO_SOT_SMD:SOT-23, F.Cu at (88.0, 89.0)
- added Q19: TSM2306, Package_TO_SOT_SMD:SOT-23, F.Cu at (91.8, 89.0)
- added Q20: TSM2306, Package_TO_SOT_SMD:SOT-23, F.Cu at (147.8, 112.0)
- added R54: 2k, Resistor_SMD:R_0805_2012Metric, F.Cu at (249.8, 115.3)
- added R55: 680, Resistor_SMD:R_0805_2012Metric, F.Cu at (223.1, 111.0)
- added R56: 100k, Resistor_SMD:R_0805_2012Metric, F.Cu at (230.0, 111.0)
- added R57: 2k, Resistor_SMD:R_0805_2012Metric, F.Cu at (185.5, 115.0)
- added R58: 2k, Resistor_SMD:R_0805_2012Metric, F.Cu at (185.5, 117.0)
- added R59: 5k, Resistor_SMD:R_0805_2012Metric, F.Cu at (245.8, 115.3)
- added R60: 10k, Resistor_SMD:R_0805_2012Metric, F.Cu at (167.5, 109.5)
- added R61: 10k, Resistor_SMD:R_0805_2012Metric, F.Cu at (163.9, 109.5)
- added R62: 10, Resistor_SMD:R_0805_2012Metric, F.Cu at (95.5, 87.5)
- added R63: 10, Resistor_SMD:R_0805_2012Metric, F.Cu at (95.5, 89.8)
- added R64: 10k, Resistor_SMD:R_0805_2012Metric, F.Cu at (151.0, 119.0)
- added R65: 10, Resistor_SMD:R_0805_2012Metric, F.Cu at (151.0, 115.5)
- added R66: 10k, Resistor_SMD:R_0805_2012Metric, F.Cu at (151.0, 112.0)
- added U20: TCMT1103, Package_SO:SOP-4_4.4x2.6mm_P1.27mm, F.Cu at (237.2, 112.2)
- added U21: CD4082, Package_SO:TSSOP-14_4.4x5mm_P0.65mm, F.Cu at (157.8, 114.5)
- added U22: LM1117-3.3, Package_TO_SOT_SMD:SOT-223-3_TabPin2, F.Cu at (250.3, 140.2)
- added U23: RFMM-0505S, MainBoard:RFMM-0505S, F.Cu at (222.9, 137.7)
- added U24: ROE-0505S, MainBoard:ROE-0505S, F.Cu at (296.8, 139.8)
- C17, C4: moved to B.Cu
- C21: value 10n -> 1u
- C23, R44: moved to F.Cu
- C27: value 1u -> 100n
- J2: value SWDebug -> SWD; footprint Connector_PinHeader_2.54mm:PinHeader_1x05_P2.54mm_Vertical -> Connector_PinHeader_2.54mm:PinHeader_2x05_P2.54mm_Vertical
- J7: value ProminentIndicator -> BYPASS_IMD; footprint Connector_Molex:Molex_Micro-Fit_3.0_43650-0215_1x02_P3.00mm_Vertical -> Connector_PinHeader_2.54mm:PinHeader_1x02_P2.54mm_Vertical
- Q16: value TSM2312 -> TSM2306
- R10: value 590 -> 10k; moved to F.Cu
- R11, R14, R33: value 100K -> 100k; moved to F.Cu
- R12: value 1M -> 10M; footprint Resistor_SMD:R_0805_2012Metric -> Resistor_SMD:R_1210_3225Metric; moved to F.Cu
- R13: value 220K -> 220k; moved to F.Cu
- R15: value 100K -> 1M; moved to F.Cu
- R16: value 10K -> 100k; moved to F.Cu
- R17: value 10K -> 1k; moved to F.Cu
- R18, R19: value 10K -> 10k; moved to F.Cu
- R2: value 1.4K -> 3.4k
- R20: value 2K2 -> PWR163S-25-1002J 10k; footprint Resistor_SMD:R_0805_2012Metric -> MainBoard:pwr163; moved to F.Cu
- R30: value 1K -> 1k; moved to F.Cu
- R31: value 3.3K -> 3.3k; moved to F.Cu
- R32: value 22K -> 22k; moved to F.Cu
- R47: value 100K -> 100k
- R51: value 1K -> 1k
- R6, R7: value 10K -> 10k
- R9: value 1.6K -> 33k; moved to F.Cu
- U12: value SN74LVC1G123 -> ADCMP350; footprint Package_SO:VSSOP-8_2.3x2mm_P0.5mm -> Package_TO_SOT_SMD:Analog_KS-4
- U13: value ISOW7841 -> TS3704IPT; footprint MainBoard:SOIC-16 -> Package_SO:TSSOP-14_4.4x5mm_P0.65mm
- U14: value LTC1865L -> Si8901; footprint Package_SO:SSOP-10_3.9x4.9mm_P1.00mm -> Package_SO:SOIC-16W_7.5x10.3mm_P1.27mm
- U16: value REF3433 -> CD4044; footprint MainBoard:SOT-23-6 -> Package_SO:TSSOP-16_4.4x5mm_P0.65mm
- U8: value LP2989 -> LM1117-3.3; footprint MainBoard:SOIC-8 -> Package_TO_SOT_SMD:SOT-223-3_TabPin2
- moved J7 229.7 mm to (142.2, 105.2)
- moved R12 169.1 mm to (309.2, 124.0)
- moved U16 159.6 mm to (157.8, 107.5), turned to 180 degrees
- moved R16 155.1 mm to (305.0, 124.0)
- moved C27 153.4 mm to (164.0, 107.5), turned to 180 degrees
- moved R17 142.6 mm to (302.5, 130.1)
- moved U13 140.4 mm to (165.7, 114.5), turned to 0 degrees
- moved R20 136.2 mm to (289.6, 91.7)
- moved C17 132.1 mm to (77.9, 128.0), turned to 180 degrees
- moved C4 127.1 mm to (77.9, 122.6), turned to 180 degrees
- moved U7 127.0 mm to (77.9, 125.3), turned to 90 degrees
- moved R8 121.9 mm to (77.9, 120.3), turned to 180 degrees
- moved J2 107.6 mm to (171.4, 93.7), turned to 90 degrees
- moved U12 103.7 mm to (306.8, 129.6)
- moved U14 92.4 mm to (237.2, 119.3), turned to 180 degrees
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Connections:
- C21 pad 1: Net-(C21-Pad1) -> +5V
- C27 pad 1: /HV/3V3ISO -> /Shutdown/1V5_REF
- C27 pad 2: -BATT -> GND
- J2 pad 1: +3V3 -> GND
- J2 pad 2: /SWDIO -> GND
- J2 pad 5: GND -> /SWDIO
- J4 pad 14: NRelayStat -> GND
- J4 pad 16: GND -> NRelayStat
- J7 pad 1: Net-(D5-Pad1) -> /IMD_Fault
- J7 pad 2: Net-(D7-Pad2) -> +12V
- K1 pad 3: +BATT -> Net-(K1-Pad3)
- K1 pad 4: Net-(K1-Pad4) -> +BATT
- Q1 pad 1: From_TSMS -> Net-(DZ3-Pad1)
- R12 pad 1: Net-(Q3-Pad3) -> Net-(R12-Pad1)
- R12 pad 2: From_SD -> +TS
- R15 pad 1: From_TSMS -> From_SD
- R15 pad 2: GND -> Net-(DZ3-Pad1)
- R16 pad 1: IMD_LED -> Net-(R12-Pad1)
- R16 pad 2: +12V -> -BATT
- R17 pad 1: Net-(Q3-Pad3) -> /HV/PROMINENT+
- R17 pad 2: Net-(Q6-Pad3) -> /HV/PROM_5V
- R19 pad 1: GND -> /HANDCART
- R19 pad 2: Net-(Q5-Pad2) -> GND
- R20 pad 1: /IMD_Fault -> Net-(K1-Pad3)
- R20 pad 2: GND -> +TS
- U12 pad 1: GND -> Net-(R12-Pad1)
- U12 pad 2: /TS_ON -> -BATT
- U12 pad 3: +3V3 -> /HV/PROMINENT-
- U12 pad 4: GND -> /HV/PROM_5V
- U13 pad 1: +3V3 -> Net-(U13-Pad1)
- U13 pad 10: /HV/5VISO -> /Shutdown/1V5_REF
- U13 pad 12: Net-(U13-Pad12) -> GND
- U13 pad 2: GND -> Net-(U13-Pad2)
- U13 pad 3: /MOSI -> +12V
- U13 pad 4: /PADC -> /Shutdown/1V5_REF
- U13 pad 5: /SCK -> /BMS_Fault
- U13 pad 6: /MISO -> /Shutdown/1V5_REF
- U13 pad 7: (no net) -> /TS_ON
- U13 pad 8: GND -> /Shutdown/1V5_REF
- U13 pad 9: -BATT -> Net-(U13-Pad9)
- U14 pad 1: Net-(U13-Pad13) -> /HV/3V3ISO
- U14 pad 10: /HV/3V3ISO -> +3V3
- U14 pad 4: Net-(U14-Pad4) -> /HV/PackV
- U14 pad 5: -BATT -> Net-(U14-Pad5)
- U14 pad 6: Net-(U13-Pad14) -> /HV/~RST~_ADCA
- U14 pad 7: Net-(U13-Pad11) -> Net-(R59-Pad2)
- U14 pad 8: Net-(U13-Pad12) -> -BATT
- U14 pad 9: Net-(U14-Pad9) -> GND
- U16 pad 1: -BATT -> Net-(U16-Pad1)
- U16 pad 2: -BATT -> (no net)
- U16 pad 3: /HV/5VISO -> Net-(U16-Pad3)
- U16 pad 4: /HV/5VISO -> Net-(U16-Pad4)
- U16 pad 5: /HV/3V3ISO -> +12V
- U16 pad 6: /HV/3V3ISO -> Net-(U13-Pad2)
- U5 pad 13: Net-(U5-Pad13) -> /RST_ADCB
- U5 pad 15: Net-(U5-Pad15) -> /6820
- U5 pad 8: /PADC -> /HANDCART
- U5 pad 9: /6820 -> Net-(U5-Pad9)
- U8 pad 1: Net-(C21-Pad1) -> GND
- U8 pad 2: (no net) -> +3V3
- U8 pad 3: GND -> +5V
Routing:
- net +3V3: track 70.4 -> 392.6 mm, vias 62 -> 32
- net +5V: track 39.0 -> 348.4 mm, vias 6 -> 5
- net -BATT: track 68.8 -> 247.9 mm, vias 16 -> 45
- net -TS: track 180.9 -> 46.2 mm, vias 3 -> 1
- net +TS: track 256.1 -> 133.7 mm, vias 2 -> 5
- net BMS_LED: track 128.0 -> 6.12 mm, vias 4 -> 0
- net /CAN-: track 141.1 -> 26.6 mm, vias 1 -> 0
- net +12V: track 24.7 -> 134.7 mm, vias 12 -> 5
- net /PADC: track 108.9 -> 0.00 mm, vias 4 -> 0
- net /CAN+: track 135.0 -> 26.6 mm, vias 1 -> 0
- net Net-(U5-Pad22): track 39.9 -> 146.5 mm, vias 2 -> 4
- net Net-(U5-Pad21): track 38.4 -> 139.9 mm, vias 2 -> 4
- net IMD_LED: track 103.0 -> 5.81 mm, vias 2 -> 0
- net Net-(DZ4-Pad1): track 92.3 -> 11.1 mm, vias 3 -> 0
- net /HV/5VISO: track 20.8 -> 98.7 mm, vias 9 -> 4
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- added copper zone on B.Cu, net +3V3
- added copper zone on B.Cu, net -BATT
- added copper zone on F.Cu, net -BATT
- added copper zone on F.Cu, net /HV/3V3ISO
- added copper zone on B.Cu, net /Shutdown/R20_heatsink
- added copper zone on F.Cu, net /Shutdown/R20_heatsink
- added copper zone on B.Cu, net GND
- removed copper zone on In1.Cu, net +12V
- removed copper zone on In1.Cu, net +3V3
- removed copper zone on In1.Cu, net +5V
- removed copper zone on In2.Cu, net -BATT
- removed copper zone on In1.Cu, net /HV/5VISO
- removed copper zone on In2.Cu, net GND
Other:
- board size 365 x 60 mm -> 292.2 x 60 mm
- copper layers 4 -> 2
- net class HV added: clearance 1.5, trace_width 0.25, via_dia 0.8, via_drill 0.4
- board text added: "5V"
- board text added: "<- Close on handcart, remove before flight."
- board text added: "Chimera BMS - MainBoard V3 2021-03-30"
- board text added: "From_TSMS"
- board text added: "SWD"
- board text added: "nc"
- board text added: "~RST~"
- board text removed: "BMS MainBoard by Gregor Gombač"
- board text removed: "MISO"
- board text removed: "MOSI"
- board text removed: "Prominent Indicator"
- board text removed: "RESET"
- board text removed: "SCK"
- board text removed: "TSMS"

Commit message: board soldered
Parts:
- removed C10, C9: 10n, Capacitor_SMD:C_0805_2012Metric
- removed R57, R58: 2k, Resistor_SMD:R_0805_2012Metric
- removed U14: Si8901, Package_SO:SOIC-16W_7.5x10.3mm_P1.27mm
- removed U17: REF2940, Package_TO_SOT_SMD:SOT-23
- removed U4: M24M02, MainBoard:SON-8
- added C24: 100n, Capacitor_SMD:C_0603_1608Metric, F.Cu at (176.2, 104.2)
- added C35: 100n, Capacitor_SMD:C_0603_1608Metric, F.Cu at (161.4, 120.2)
- added J13: SWD_old, Connector_PinHeader_2.54mm:PinHeader_1x06_P2.54mm_Vertical, F.Cu at (242.8, 88.7)
- added R21: 22, Resistor_SMD:R_0805_2012Metric, F.Cu at (222.4, 119.2)
- added R22: 10k, Resistor_SMD:R_0805_2012Metric, F.Cu at (141.3, 115.2)
- added R23: 100k, Resistor_SMD:R_0805_2012Metric, F.Cu at (159.4, 96.2)
- added R24: 1k, Resistor_SMD:R_0805_2012Metric, F.Cu at (251.7, 115.5)
- added REF**: MountingHole_4.3mm_M4, MountingHole:MountingHole_4.3mm_M4, F.Cu at (264.8, 140.4)
- added SW1: RESET, Button_Switch_SMD:SW_SPST_FSMSM, F.Cu at (182.3, 106.1)
- added SW2: SD_RESET, Button_Switch_SMD:SW_SPST_FSMSM, F.Cu at (161.4, 123.3)
- C11, C13, C15, C17, C19, C20, C26, C27, C28, C29, C3, C30, C4, C7: footprint Capacitor_SMD:C_0805_2012Metric -> Capacitor_SMD:C_0603_1608Metric
- C14, C6, C8: value 10n -> 100n; footprint Capacitor_SMD:C_0805_2012Metric -> Capacitor_SMD:C_0603_1608Metric
- C18, C22: value 47n -> 100n; footprint Capacitor_SMD:C_0805_2012Metric -> Capacitor_SMD:C_0603_1608Metric
- Q17: value IRLML0100TRPbF -> DMN10H220L-7
- R13: value 220k -> 100k
- R19: value 10k -> 22
- R31: value 3.3k -> 22
- R33: value 100k -> 10k
- R54: value 2k -> 1k
- R55: value 680 -> 1k
- R59: value 5k -> 1k
- R62, R63, R65: value 10 -> 22
- R9: value 33k -> 22k
- U15: footprint MainBoard:MSOP-8 -> MainBoard:MSOP-8_and_TSOT-23-8
- U3: value M24M02 -> Si8900; footprint MainBoard:SON-8 -> MainBoard:SOIC-16
- moved C6 67.3 mm to (256.3, 137.6), turned to 0 degrees
- moved U3 46.9 mm to (237.2, 119.3), turned to 90 degrees
- moved R19 40.9 mm to (222.4, 121.3), turned to 180 degrees
- moved R51 32.5 mm to (228.9, 95.3), turned to 270 degrees
- moved C28 12.7 mm to (261.7, 117.0)
- moved G*** 5.21 mm to (154.4, 131.8)
- moved C15 4.73 mm to (227.9, 115.2)
- moved C16 4.22 mm to (223.4, 115.1)
- moved D2 3.30 mm to (256.9, 96.2)
- moved R14 2.92 mm to (161.4, 96.2)
- moved R10 2.24 mm to (141.3, 118.7)
- moved R9 1.26 mm to (141.3, 111.7)
- moved C8 0.69 mm to (212.7, 128.0)
- moved R54 0.30 mm to (249.6, 115.5), turned to 90 degrees
- moved R3 0.28 mm to (244.4, 126.4)
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Connections:
- C28 pad 1: /HV/4VISO -> /HV/5VISO
- C6 pad 1: +3V3 -> /HV/3V3ISO
- C6 pad 2: GND -> -BATT
- J11 pad 2: +3V3 -> GND
- J2 pad 10: Net-(J2-Pad10) -> /RX
- J2 pad 9: Net-(J2-Pad9) -> /TX
- R18 pad 1: Net-(R13-Pad2) -> Net-(R18-Pad1)
- R19 pad 1: /HANDCART -> Net-(R19-Pad1)
- R19 pad 2: GND -> /ADC_RX
- R54 pad 1: /HV/3V3ISO -> /HV/~RST~_ADCA
- R54 pad 2: /HV/~RST~_ADCA -> Net-(R24-Pad1)
- R9 pad 2: /IMD -> Net-(R22-Pad1)
- U11 pad 3: Net-(R13-Pad2) -> Net-(R18-Pad1)
- U15 pad 8: /HV/4VISO -> /HV/5VISO
- U3 pad 1: (no net) -> /HV/3V3ISO
- U3 pad 2: (no net) -> Net-(U3-Pad2)
- U3 pad 3: GND -> /HV/TSV
- U3 pad 4: GND -> /HV/PackV
- U3 pad 5: /SDA -> Net-(U3-Pad5)
- U3 pad 6: /SCL -> /HV/~RST~_ADCA
- U3 pad 7: /WC -> Net-(R59-Pad2)
- U3 pad 8: +3V3 -> -BATT
- U5 pad 2: Net-(U5-Pad2) -> /HANDCART
- U5 pad 29: /SCL -> /ADC_RX
- U5 pad 30: /SDA -> /ADC_TX
- U5 pad 8: /HANDCART -> /TX
- U5 pad 9: Net-(U5-Pad9) -> /RX
Routing:
- net /RST: track 44.8 -> 140.9 mm, vias 1 -> 3
- net /SWCLK: track 48.3 -> 131.8 mm, vias 1 -> 2
- net /SWDIO: track 49.8 -> 127.3 mm, vias 1 -> 2
- net /SCL: track 72.6 -> 0.00 mm, vias 6 -> 0
- net /SDA: track 68.5 -> 0.00 mm, vias 4 -> 0
- net +5V: track 348.4 -> 412.5 mm
- net /RX: track 0.00 -> 47.7 mm, vias 0 -> 3
- net /TX: track 0.00 -> 43.4 mm, vias 0 -> 3
- net RESET_BUTTON: track 88.0 -> 129.1 mm, vias 1 -> 2
- net /ADC_TX: track 0.00 -> 37.0 mm
- net /ADC_RX: track 0.00 -> 36.9 mm
- net /WC: track 31.4 -> 0.00 mm
- net +3V3: track 392.6 -> 366.9 mm, vias 32 -> 30
- net /HV/5VISO: track 98.7 -> 118.8 mm, vias 4 -> 6
- net /HV/4VISO: track 17.8 -> 0.00 mm, vias 2 -> 0
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Other:
- rule via_min_size: 0.4 -> 0.6
- board text added: "<- IMD_Fault BYPASS"
- board text added: "MCU_RESET"
- board text added: "Muletto Evoluzione"
- board text added: "RX"
- board text added: "SD_RESET"
- board text added: "SWD_old"
- board text added: "TX"
