File: mainboard/MainBoard.sch (KiCad schematic (older format))
At the start: 52 parts, among them J1 isoSPI, J11 ON_HANDCART, J3 IMD, J4 IO, U1 LTC6820, U10 REF2920, U2 HM2103, U3 M24M02, U4 M24M02, U5 STM32F334K8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

Commit message: finished footprint association
Parts:
- C21: value 1uF -> 1u
- C24: renamed from C?; value 10uF -> 4.7u
- J11: footprint (none) -> MainBoard:PinHeader_1x02_P3mm_Vertical
- J2: renamed from J?; footprint (none) -> Connector_PinHeader_2.54mm:PinHeader_2x05_P2.54mm_Vertical
- R19: renamed from 10k1; value R -> 10k; footprint (none) -> Resistor_SMD:R_0805_2012Metric
- R2: value 1.4K -> 3.4k
- R51: value 1K -> 1k
- R6, R7: value 10K -> 10k
- U8: renamed from U?; footprint (none) -> Package_TO_SOT_SMD:SOT-223-3_TabPin2
Changed lines of the file:
@@
 P 9450 1150
 F 0 "R2" V 9350 1150 50  0000 C CNN
-F 1 "1.4K" V 9450 1150 50  0000 C CNN
+F 1 "3.4k" V 9450 1150 50  0000 C CNN
 F 2 "Resistor_SMD:R_0805_2012Metric" V 9380 1150 50  0001 C CNN
 F 3 "~" H 9450 1150 50  0001 C CNN
@@
 P 8700 5550
 F 0 "C21" V 8550 5550 50  0000 C CNN
-F 1 "1uF" V 8850 5550 50  0000 C CNN
+F 1 "1u" V 8850 5550 50  0000 C CNN
 F 2 "Capacitor_SMD:C_0805_2012Metric" H 8738 5400 50  0001 C CNN
 F 3 "~" H 8700 5550 50  0001 C CNN
@@
 P 6400 3150
 F 0 "R7" V 6300 3150 50  0000 C CNN
-F 1 "10K" V 6400 3150 50  0000 C CNN
+F 1 "10k" V 6400 3150 50  0000 C CNN
 F 2 "Resistor_SMD:R_0805_2012Metric" V 6330 3150 50  0001 C CNN
 F 3 "~" H 6400 3150 50  0001 C CNN
@@
 P 6650 2900
 F 0 "R6" V 6550 2900 50  0000 C CNN
-F 1 "10K" V 6650 2900 50  0000 C CNN
+F 1 "10k" V 6650 2900 50  0000 C CNN
 F 2 "Resistor_SMD:R_0805_2012Metric" V 6580 2900 50  0001 C CNN
 F 3 "~" H 6650 2900 50  0001 C CNN
@@
 P 4100 3300
 F 0 "R51" V 4200 3300 50  0000 C CNN
-F 1 "1K" V 4100 3300 50  0000 C CNN
+F 1 "1k" V 4100 3300 50  0000 C CNN
 F 2 "Resistor_SMD:R_0805_2012Metric" V 4030 3300 50  0001 C CNN
 F 3 "~" H 4100 3300 50  0001 C CNN
@@
 HANDCART
 $Comp
-L Device:R 10k1
+L Device:R R19
 U 1 1 6050CC83
 P 10300 2850
-F 0 "10k1" V 10300 2850 50  0000 C CNN
-F 1 "R" V 10400 2850 50  0000 C CNN
-F 2 "" V 10230 2850 50  0001 C CNN
+F 0 "R19" V 10400 2850 50  0000 C CNN
+F 1 "10k" V 10300 2850 50  0000 C CNN
+F 2 "Resistor_SMD:R_0805_2012Metric" V 10230 2850 50  0001 C CNN
 F 3 "~" H 10300 2850 50  0001 C CNN
 	1    10300 2850
@@
 F 0 "J11" H 10780 2742 50  0000 L CNN
 F 1 "ON_HANDCART" H 10500 2850 50  0000 L CNN
-F 2 "" H 10700 2750 50  0001 C CNN
+F 2 "MainBoard:PinHeader_1x02_P3mm_Vertical" H 10700 2750 50  0001 C CNN
 F 3 "~" H 10700 2750 50  0001 C CNN
 	1    10700 2750
@@
 CHECK: unpopulated
 $Comp
-L Connector_Generic:Conn_02x05_Odd_Even J?
+L Connector_Generic:Conn_02x05_Odd_Even J2
 U 1 1 606179E7
 P 9050 2900
-F 0 "J?" H 9100 3317 50  0000 C CNN
+F 0 "J2" H 9100 3317 50  0000 C CNN
 F 1 "SWD" H 9100 3226 50  0000 C CNN
-F 2 "" H 9050 2900 50  0001 C CNN
+F 2 "Connector_PinHeader_2.54mm:PinHeader_2x05_P2.54mm_Vertical" H 9050 2900 50  0001 C CNN
 F 3 "~" H 9050 2900 50  0001 C CNN
 	1    9050 2900
@@
 	8450 2900 8850 2900
 $Comp
-L power:+5V #PWR?
+L power:+5V #PWR049
 U 1 1 6073E490
 P 9450 3000
-F 0 "#PWR?" H 9450 2850 50  0001 C CNN
+F 0 "#PWR049" H 9450 2850 50  0001 C CNN
 F 1 "+5V" V 9450 3150 50  0000 L CNN
 F 2 "" H 9450 3000 50  0001 C CNN
@@
 	9350 2700 9450 2700
 $Comp
-L power:GND #PWR?
+L power:GND #PWR048
 U 1 1 60784403
 P 9450 2700
-F 0 "#PWR?" H 9450 2450 50  0001 C CNN
+F 0 "#PWR048" H 9450 2450 50  0001 C CNN
 F 1 "GND" V 9450 2550 50  0000 R CNN
 F 2 "" H 9450 2700 50  0001 C CNN
@@
 	8350 2400 8350 3200
 $Comp
-L Regulator_Linear:LM1117-3.3 U?
+L Regulator_Linear:LM1117-3.3 U8
 U 1 1 608FC0D4
 P 9100 5300
-F 0 "U?" H 9100 5542 50  0000 C CNN
+F 0 "U8" H 9100 5542 50  0000 C CNN
 F 1 "LM1117-3.3" H 9100 5451 50  0000 C CNN
-F 2 "" H 9100 5300 50  0001 C CNN
+F 2 "Package_TO_SOT_SMD:SOT-223-3_TabPin2" H 9100 5300 50  0001 C CNN
 F 3 "http://www.ti.com/lit/ds/symlink/lm1117.pdf" H 9100 5300 50  0001 C CNN
 	1    9100 5300
@@
 Connection ~ 8700 5300
 $Comp
-L Device:C C?
+L Device:C C24
 U 1 1 60989FBB
 P 9500 5550
-F 0 "C?" V 9350 5550 50  0000 C CNN
-F 1 "10uF" V 9650 5550 50  0000 C CNN
+F 0 "C24" V 9350 5550 50  0000 C CNN
+F 1 "4.7u" V 9650 5550 50  0000 C CNN
 F 2 "Capacitor_SMD:C_0805_2012Metric" H 9538 5400 50  0001 C CNN
 F 3 "~" H 9500 5550 50  0001 C CNN
@@
 	9500 5300 9650 5300
 $Comp
-L power:GND #PWR?
+L power:GND #PWR064
 U 1 1 60A549B3
 P 9500 5800
-F 0 "#PWR?" H 9500 5550 50  0001 C CNN
+F 0 "#PWR064" H 9500 5550 50  0001 C CNN
 F 1 "GND" H 9500 5650 50  0000 C CNN
 F 2 "" H 9500 5800 50  0001 C CNN

Commit message: Done early board
Parts:
- removed C24: 4.7u, Capacitor_SMD:C_0805_2012Metric, symbol Device:C
- added J7: BYPASS_IMD, Connector_PinHeader_2.54mm:PinHeader_1x02_P2.54mm_Vertical, symbol Connector_Generic:Conn_01x02
- J11: footprint MainBoard:PinHeader_1x02_P3mm_Vertical -> Connector_PinHeader_2.54mm:PinHeader_1x02_P2.54mm_Vertical
Connections:
- net +12V: now also J7.2 (Pin_2)
- net GND: now also J4.14 (Pin_14); no longer J4.16 (Pin_16)
- net IMD_Fault: now also J7.1 (Pin_1)
- net NRelayStat: now also J4.16 (Pin_16); no longer J4.14 (Pin_14)
Other:
- note added: "Close this contact to bypass \nin case of no IMD present."
- moved on the sheet: J3, R10, R9
Changed lines of the file:
@@
 encoding utf-8
 Sheet 1 3
-Title "Chimera BMS"
-Date "2021-03-28"
+Title "Chimera BMS - MainBoard"
+Date "2021-03-29"
 Rev "V3"
 Comp "E-Agle TRT"
@@
 L Connector_Generic:Conn_01x08 J3
 U 1 1 5B191837
-P 2000 5200
-F 0 "J3" H 2000 5600 50  0000 C CNN
-F 1 "IMD" V 2100 5150 50  0000 C CNN
-F 2 "MainBoard:PinHeader_1x08_P3mm_Vertical" H 2000 5200 50  0001 C CNN
-F 3 "https://www.bender.de/fileadmin/content/Products/d/e/IR155-32xx-V004_D00115_D_XXEN.pdf" H 2000 5200 50  0001 C CNN
-	1    2000 5200
-	1    0    0    -1
-$EndComp
-Wire Wire Line
-	1800 4900 1700 4900
+P 2000 4750
+F 0 "J3" H 2000 5150 50  0000 C CNN
+F 1 "IMD" V 2100 4700 50  0000 C CNN
+F 2 "MainBoard:PinHeader_1x08_P3mm_Vertical" H 2000 4750 50  0001 C CNN
+F 3 "https://www.bender.de/fileadmin/content/Products/d/e/IR155-32xx-V004_D00115_D_XXEN.pdf" H 2000 4750 50  0001 C CNN
+	1    2000 4750
+	1    0    0    -1
+$EndComp
+Wire Wire Line
+	1800 4450 1700 4450
 $Comp
 L power:GND #PWR038
 U 1 1 5B1CEF4A
-P 1700 4900
-F 0 "#PWR038" H 1700 4650 50  0001 C CNN
-F 1 "GND" V 1700 4750 50  0000 R CNN
-F 2 "" H 1700 4900 50  0001 C CNN
-F 3 "" H 1700 4900 50  0001 C CNN
-	1    1700 4900
-	0    1    1    0
-$EndComp
-Wire Wire Line
-	1800 5100 1700 5100
-Wire Wire Line
-	1800 5200 1700 5200
-Wire Wire Line
-	1700 5000 1800 5000
-NoConn ~ 1800 5500
-Text Label 1400 5600 0    50   ~ 0
+P 1700 4450
+F 0 "#PWR038" H 1700 4200 50  0001 C CNN
+F 1 "GND" V 1700 4300 50  0000 R CNN
+F 2 "" H 1700 4450 50  0001 C CNN
+F 3 "" H 1700 4450 50  0001 C CNN
+	1    1700 4450
+	0    1    1    0
+$EndComp
+Wire Wire Line
+	1800 4650 1700 4650
+Wire Wire Line
+	1800 4750 1700 4750
+Wire Wire Line
+	1700 4550 1800 4550
+NoConn ~ 1800 5050
+Text Label 1400 5150 0    50   ~ 0
 IMD_Fault
 Wire Wire Line
-	1400 5600 1800 5600
-NoConn ~ 1800 5400
+	1400 5150 1800 5150
+NoConn ~ 1800 4950
 $Comp
 L power:GND #PWR044
 U 1 1 5B541514
-P 1700 5200
-F 0 "#PWR044" H 1700 4950 50  0001 C CNN
-F 1 "GND" V 1700 5050 50  0000 R CNN
-F 2 "" H 1700 5200 50  0001 C CNN
-F 3 "" H 1700 5200 50  0001 C CNN
-	1    1700 5200
+P 1700 4750
+F 0 "#PWR044" H 1700 4500 50  0001 C CNN
+F 1 "GND" V 1700 4600 50  0000 R CNN
+F 2 "" H 1700 4750 50  0001 C CNN
+F 3 "" H 1700 4750 50  0001 C CNN
+	1    1700 4750
 	0    1    1    0
 $EndComp
@@
 L power:GND #PWR042
 U 1 1 5B54160F
-P 1700 5100
-F 0 "#PWR042" H 1700 4850 50  0001 C CNN
-F 1 "GND" V 1700 4950 50  0000 R CNN
-F 2 "" H 1700 5100 50  0001 C CNN
-F 3 "" H 1700 5100 50  0001 C CNN
-	1    1700 5100
+P 1700 4650
+F 0 "#PWR042" H 1700 4400 50  0001 C CNN
+F 1 "GND" V 1700 4500 50  0000 R CNN
+F 2 "" H 1700 4650 50  0001 C CNN
+F 3 "" H 1700 4650 50  0001 C CNN
+	1    1700 4650
 	0    1    1    0
 $EndComp
@@
 L power:+12V #PWR039
 U 1 1 5B541F7A
-P 1700 5000
-F 0 "#PWR039" H 1700 4850 50  0001 C CNN
-F 1 "+12V" V 1700 5150 50  0000 L CNN
-F 2 "" H 1700 5000 50  0001 C CNN
-F 3 "" H 1700 5000 50  0001 C CNN
-	1    1700 5000
+P 1700 4550
+F 0 "#PWR039" H 1700 4400 50  0001 C CNN
+F 1 "+12V" V 1700 4700 50  0000 L CNN
+F 2 "" H 1700 4550 50  0001 C CNN
+F 3 "" H 1700 4550 50  0001 C CNN
+	1    1700 4550
 	0    -1   -1   0
 $EndComp
@@
 IMD
 Wire Wire Line
-	1000 5300 1000 5400
+	1000 4850 1000 4950
 $Comp
 L Device:R R10
 U 1 1 5B4093B7
-P 1000 5550
-F 0 "R10" V 900 5550 50  0000 C CNN
-F 1 "10k" V 1000 5550 50  0000 C CNN
-F 2 "Resistor_SMD:R_0805_2012Metric" V 930 5550 50  0001 C CNN
-F 3 "~" H 1000 5550 50  0001 C CNN
-	1    1000 5550
-	1    0    0    -1
-$EndComp
-Wire Wire Line
-	1000 5700 1000 5800
+P 1000 5100
+F 0 "R10" V 900 5100 50  0000 C CNN
+F 1 "10k" V 1000 5100 50  0000 C CNN
+F 2 "Resistor_SMD:R_0805_2012Metric" V 930 5100 50  0001 C CNN
+F 3 "~" H 1000 5100 50  0001 C CNN
+	1    1000 5100
+	1    0    0    -1
+$EndComp
+Wire Wire Line
+	1000 5250 1000 5350
 $Comp
 L power:GND #PWR050
 U 1 1 5B42E62A
-P 1000 5800
-F 0 "#PWR050" H 1000 5550 50  0001 C CNN
-F 1 "GND" H 1000 5650 50  0000 C CNN
-F 2 "" H 1000 5800 50  0001 C CNN
-F 3 "" H 1000 5800 50  0001 C CNN
-	1    1000 5800
+P 1000 5350
+F 0 "#PWR050" H 1000 5100 50  0001 C CNN
+F 1 "GND" H 1000 5200 50  0000 C CNN
+F 2 "" H 1000 5350 50  0001 C CNN
+F 3 "" H 1000 5350 50  0001 C CNN
+	1    1000 5350
 	1    0    0    -1
 $EndComp
@@
 L Device:R R9
 U 1 1 5B45397A
-P 1250 5300
-F 0 "R9" V 1150 5300 50  0000 C CNN
-F 1 "33k" V 1250 5300 50  0000 C CNN
-F 2 "Resistor_SMD:R_0805_2012Metric" V 1180 5300 50  0001 C CNN
-F 3 "~" H 1250 5300 50  0001 C CNN
-	1    1250 5300
-	0    1    1    0
-$EndComp
-Wire Wire Line
-	1000 5300 1100 5300
-Wire Wire Line
-	1400 5300 1800 5300
-Wire Wire Line
-	1000 5300 800  5300
-Connection ~ 1000 5300
-Text Label 800  5300 0    50   ~ 0
+P 1250 4850
+F 0 "R9" V 1150 4850 50  0000 C CNN
+F 1 "33k" V 1250 4850 50  0000 C CNN
+F 2 "Resistor_SMD:R_0805_2012Metric" V 1180 4850 50  0001 C CNN
+F 3 "~" H 1250 4850 50  0001 C CNN
+	1    1250 4850
+	0    1    1    0
+$EndComp
+Wire Wire Line
+	1000 4850 1100 4850
+Wire Wire Line
+	1400 4850 1800 4850
+Wire Wire Line
+	1000 4850 800  4850
+Connection ~ 1000 4850
+Text Label 800  4850 0    50   ~ 0
 IMD
 NoConn ~ 4600 3950
@@
 Text GLabel 1750 6850 2    50   Input ~ 0
 RelayStat
-Text GLabel 1750 7150 2    50   Input ~ 0
+Text GLabel 1750 7250 2    50   Input ~ 0
 NRelayStat
 $Comp
@@
 	1150 7250 1050 7250
 Wire Wire Line
-	1650 7250 1750 7250
+	1650 7150 1750 7150
 $Comp
 L power:GND #PWR059
@@
 L power:GND #PWR060
 U 1 1 5BC6DE63
-P 1750 7250
-F 0 "#PWR060" H 1750 7000 50  0001 C CNN
-F 1 "GND" V 1750 7100 50  0000 R CNN
-F 2 "" H 1750 7250 50  0001 C CNN
-F 3 "" H 1750 7250 50  0001 C CNN
-	1    1750 7250
+P 1750 7150
+F 0 "#PWR060" H 1750 6900 50  0001 C CNN
+F 1 "GND" V 1750 7000 50  0000 R CNN
+F 2 "" H 1750 7150 50  0001 C CNN
+F 3 "" H 1750 7150 50  0001 C CNN
+	1    1750 7150
 	0    -1   -1   0
 $EndComp
@@
 	950  7150 1150 7150
 Wire Wire Line
-	1650 7150 1750 7150
+	1650 7250 1750 7250
 $Sheet
 S 3100 5150 900  700
@@
 F 0 "J11" H 10780 2742 50  0000 L CNN
 F 1 "ON_HANDCART" H 10500 2850 50  0000 L CNN
-F 2 "MainBoard:PinHeader_1x02_P3mm_Vertical" H 10700 2750 50  0001 C CNN
+F 2 "Connector_PinHeader_2.54mm:PinHeader_1x02_P2.54mm_Vertical" H 10700 2750 50  0001 C CNN
 F 3 "~" H 10700 2750 50  0001 C CNN
 	1    10700 2750
@@
 	9850 3200 11150 3200
 NoConn ~ 5800 3200
-Text Notes 1400 5850 0    50   ~ 0
+Text Notes 1400 5400 0    50   ~ 0
 12V CMOS\nHIGH: OK\nLOW: fault
 Text Notes 600  4200 0    50   ~ 0
@@
 Connection ~ 8700 5300
 $Comp
-L Device:C C24
-U 1 1 60989FBB
-P 9500 5550
-F 0 "C24" V 9350 5550 50  0000 C CNN
-F 1 "4.7u" V 9650 5550 50  0000 C CNN
-F 2 "Capacitor_SMD:C_0805_2012Metric" H 9538 5400 50  0001 C CNN
-F 3 "~" H 9500 5550 50  0001 C CNN
-	1    9500 5550
-	1    0    0    -1
-$EndComp
-$Comp
 L power:+3.3V #PWR046
 U 1 1 5AF3CEC7
@@
 	8600 5300 8700 5300
 Wire Wire Line
-	9400 5300 9500 5300
-Wire Wire Line
-	9500 5400 9500 5300
-Connection ~ 9500 5300
-Wire Wire Line
-	9500 5300 9650 5300
-$Comp
-L power:GND #PWR064
-U 1 1 60A549B3
-P 9500 5800
-F 0 "#PWR064" H 9500 5550 50  0001 C CNN
-F 1 "GND" H 9500 5650 50  0000 C CNN
-F 2 "" H 9500 5800 50  0001 C CNN
-F 3 "" H 9500 5800 50  0001 C CNN
-	1    9500 5800
-	1    0    0    -1
-$EndComp
-Wire Wire Line
 	9100 5600 9100 5800
 Wire Wire Line
-	9500 5700 9500 5800
+	9400 5300 9650 5300
+$Comp
+L Connector_Generic:Conn_01x02 J7
+U 1 1 60675482
+P 2000 5550
+F 0 "J7" H 2080 5542 50  0000 L CNN
+F 1 "BYPASS_IMD" H 2080 5451 50  0000 L CNN
+F 2 "Connector_PinHeader_2.54mm:PinHeader_1x02_P2.54mm_Vertical" H 2000 5550 50  0001 C CNN
+F 3 "~" H 2000 5550 50  0001 C CNN
+	1    2000 5550
+	1    0    0    -1
+$EndComp
+Text Label 1400 5550 0    50   ~ 0
+IMD_Fault
+Wire Wire Line
+	1400 5550 1800 5550
+$Comp
+L power:+12V #PWR064
+U 1 1 6068C359
+P 1750 5650
+F 0 "#PWR064" H 1750 5500 50  0001 C CNN
+F 1 "+12V" V 1750 5800 50  0000 L CNN
+F 2 "" H 1750 5650 50  0001 C CNN
+F 3 "" H 1750 5650 50  0001 C CNN
+	1    1750 5650
+	0    -1   -1   0
+$EndComp
+Wire Wire Line
+	1750 5650 1800 5650
+Text Notes 1350 5850 0    50   ~ 0
+Close this contact to bypass \nin case of no IMD present.
 $EndSCHEMATC

Commit message: board soldered
Parts:
- removed C10, C6, C9: 10n, Capacitor_SMD:C_0805_2012Metric, symbol Device:C
- removed R19: 10k, Resistor_SMD:R_0805_2012Metric, symbol Device:R
- removed R57, R58: 2k, Resistor_SMD:R_0805_2012Metric, symbol Device:R
- removed U3, U4: M24M02, MainBoard:SON-8, symbol MainBoard:M24M02
- added C24, C35: 100n, Capacitor_SMD:C_0603_1608Metric, symbol Device:C
- added J13: SWD_old, Connector_PinHeader_2.54mm:PinHeader_1x06_P2.54mm_Vertical, symbol Connector_Generic:Conn_01x06
- added R22: 10k, Resistor_SMD:R_0805_2012Metric, symbol Device:R
- added SW1: RESET, Button_Switch_SMD:SW_SPST_FSMSM, symbol Switch:SW_Push
- added SW2: SD_RESET, Button_Switch_SMD:SW_SPST_FSMSM, symbol Switch:SW_Push
- C11, C15, C17, C20, C3, C4, C7: footprint Capacitor_SMD:C_0805_2012Metric -> Capacitor_SMD:C_0603_1608Metric
- C14, C8: value 10n -> 100n; footprint Capacitor_SMD:C_0805_2012Metric -> Capacitor_SMD:C_0603_1608Metric
- C18, C22: value 47n -> 100n; footprint Capacitor_SMD:C_0805_2012Metric -> Capacitor_SMD:C_0603_1608Metric
- R4: value 100 -> 120
- R9: value 33k -> 22k
Connections:
- net +3V3: now also J13.2 (Pin_2); no longer J11.2 (Pin_2)
- net +5V: now also J13.1 (Pin_1)
- net GND: now also J11.2 (Pin_2), C24.2, C35.2, J13.6 (Pin_6), SW1.1, SW2.1
- net HANDCART: now also U5.2 (PF0); no longer U5.8 (PA2)
- net IMD: now also R22.2; no longer R9.2
- net RESET_BUTTON: now also C35.1, SW2.2
- net RST: now also C24.1, J13.5 (Pin_5), SW1.2
- net SWCLK: now also J13.4 (Pin_4)
- net SWDIO: now also J13.3 (Pin_3)
- net RX: now reaches U5.9 (PA3)
- net RX: now also J2.10 (Pin_10)
- net TX: now reaches J2.9 (Pin_9)
- net TX: now also U5.8 (PA2)
- net SCL renamed ADC_RX
- net SDA renamed ADC_TX
- new net: R22.1, R9.2
- no-connect marks 10 -> 6
Other:
- note removed: "CHECK: unpopulated"
- moved on the sheet: C1, C18, R10, R9, U6

Commit message: corrected pulldown and air+ mosfet driving
Parts:
- added R25, R26, R27: 100k, Resistor_SMD:R_0805_2012Metric, symbol Device:R
Connections:
- net BMS_Fault: now also R26.1
- net GND: now also R25.2, R26.2, R27.2
- net PC_Ended: now also R27.1
- net TS_ON: now also R25.1
Changed lines of the file:
@@
 Wire Wire Line
 	2700 550  3500 550
+$Comp
+L Device:R R?
+U 1 1 60A2180C
+P 6850 5450
+AR Path="/5B045B0D/60A2180C" Ref="R?"  Part="1"
+AR Path="/60A2180C" Ref="R25"  Part="1"
+F 0 "R25" V 6750 5450 50  0000 C CNN
+F 1 "100k" V 6850 5450 50  0000 C CNN
+F 2 "Resistor_SMD:R_0805_2012Metric" V 6780 5450 50  0001 C CNN
+F 3 "~" H 6850 5450 50  0001 C CNN
+	1    6850 5450
+	1    0    0    -1
+$EndComp
+$Comp
+L Device:R R?
+U 1 1 60A3611C
+P 7050 5450
+AR Path="/5B045B0D/60A3611C" Ref="R?"  Part="1"
+AR Path="/60A3611C" Ref="R26"  Part="1"
+F 0 "R26" V 6950 5450 50  0000 C CNN
+F 1 "100k" V 7050 5450 50  0000 C CNN
+F 2 "Resistor_SMD:R_0805_2012Metric" V 6980 5450 50  0001 C CNN
+F 3 "~" H 7050 5450 50  0001 C CNN
+	1    7050 5450
+	1    0    0    -1
+$EndComp
+$Comp
+L power:GND #PWR022
+U 1 1 60A4A952
+P 6850 5600
+F 0 "#PWR022" H 6850 5350 50  0001 C CNN
+F 1 "GND" V 6850 5450 50  0000 R CNN
+F 2 "" H 6850 5600 50  0001 C CNN
+F 3 "" H 6850 5600 50  0001 C CNN
+	1    6850 5600
+	1    0    0    -1
+$EndComp
+$Comp
+L power:GND #PWR023
+U 1 1 60A4AE02
+P 7050 5600
+F 0 "#PWR023" H 7050 5350 50  0001 C CNN
+F 1 "GND" V 7050 5450 50  0000 R CNN
+F 2 "" H 7050 5600 50  0001 C CNN
+F 3 "" H 7050 5600 50  0001 C CNN
+	1    7050 5600
+	1    0    0    -1
+$EndComp
+Text Label 6850 4900 3    50   ~ 0
+TS_ON
+Text Label 7050 4900 3    50   ~ 0
+BMS_Fault
+Wire Wire Line
+	7050 4900 7050 5300
+Wire Wire Line
+	6850 5300 6850 4900
+Text Label 7250 4900 3    50   ~ 0
+PC_Ended
+$Comp
+L Device:R R?
+U 1 1 60A7560C
+P 7250 5450
+AR Path="/5B045B0D/60A7560C" Ref="R?"  Part="1"
+AR Path="/60A7560C" Ref="R27"  Part="1"
+F 0 "R27" V 7150 5450 50  0000 C CNN
+F 1 "100k" V 7250 5450 50  0000 C CNN
+F 2 "Resistor_SMD:R_0805_2012Metric" V 7180 5450 50  0001 C CNN
+F 3 "~" H 7250 5450 50  0001 C CNN
+	1    7250 5450
+	1    0    0    -1
+$EndComp
+Wire Wire Line
+	7250 4900 7250 5300
+$Comp
+L power:GND #PWR025
+U 1 1 60AB414D
+P 7250 5600
+F 0 "#PWR025" H 7250 5350 50  0001 C CNN
+F 1 "GND" V 7250 5450 50  0000 R CNN
+F 2 "" H 7250 5600 50  0001 C CNN
+F 3 "" H 7250 5600 50  0001 C CNN
+	1    7250 5600
+	1    0    0    -1
+$EndComp
 $EndSCHEMATC
